Commit message: Added ffw_bh5_rev1 launch file
Signed-off-by: Hyunwoo Nam <nhw@robotis.com>

File: ffw_description/urdf/common/rh_5_right/rh_5_right.urdf.xacro (robot description, xacro)
@@ -1,7 +1,12 @@
 <?xml version="1.0" encoding="UTF-8"?>
-<robot xmlns:xacro="http://www.ros.org/wiki/xacro" name="robotis_hand">
-   <xacro:macro name="robotis_hand" params="prefix">
+<robot xmlns:xacro="http://www.ros.org/wiki/xacro">
+   <xacro:macro name="rh_5_right" params="prefix parent *origin">
       <xacro:property name="meshes_file_direction" value="package://ffw_description/meshes/common/rh_5_right/" />
-      <link name="${prefix}robotis_hand_base">
+      <joint name="${prefix}joint" type="fixed">
+         <xacro:insert_block name="origin" />
+         <parent link="${parent}"/>
+         <child link="${prefix}rh_5_right_base" />
+      </joint>
+      <link name="${prefix}rh_5_right_base">
          <visual>
             <origin xyz="0 0 0" rpy="0 0 0" />
@@ -31,7 +36,7 @@
       </link>
       <!-- THUMB -->
-      <joint name="${prefix}finger_joint_1" type="revolute">
-         <parent link="${prefix}robotis_hand_base" />
-         <child link="${prefix}finger_link_1" />
+      <joint name="${prefix}finger_r_joint1" type="revolute">
+         <parent link="${prefix}rh_5_right_base" />
+         <child link="${prefix}finger_r_link1" />
          <origin xyz="0.0145 0.02624 0.05394" rpy="-0.523599 0 0" />
          <axis xyz="0 0 1" />
@@ -39,5 +44,5 @@
          <dynamics damping="0.05" />
       </joint>
-      <link name="${prefix}finger_link_1">
+      <link name="${prefix}finger_r_link1">
          <visual>
             <origin xyz="0 0 0" rpy="0 0 0" />
@@ -66,7 +71,7 @@
          </inertial>
       </link>
-      <joint name="${prefix}finger_joint_2" type="revolute">
-         <parent link="${prefix}finger_link_1" />
-         <child link="${prefix}finger_link_2" />
+      <joint name="${prefix}finger_r_joint2" type="revolute">
+         <parent link="${prefix}finger_r_link1" />
+         <child link="${prefix}finger_r_link2" />
          <origin xyz="0.0 0.028 0.0" rpy="0.523599 0 0" />
          <axis xyz="1 0 0" />
@@ -74,5 +79,5 @@
          <dynamics damping="0.05" />
       </joint>
-      <link name="${prefix}finger_link_2">
+      <link name="${prefix}finger_r_link2">
          <visual>
             <origin xyz="0 0 0" rpy="0 0 0" />
@@ -101,7 +106,7 @@
          </inertial>
       </link>
-      <joint name="${prefix}finger_joint_3" type="revolute">
-         <parent link="${prefix}finger_link_2" />
-         <child link="${prefix}finger_link_3" />
+      <joint name="${prefix}finger_r_joint3" type="revolute">
+         <parent link="${prefix}finger_r_link2" />
+         <child link="${prefix}finger_r_link3" />
          <origin xyz="0.0 0.0145 0.035" rpy="0 0 0" />
          <axis xyz="0 1 0" />
@@ -109,5 +114,5 @@
          <dynamics damping="0.05" />
       </joint>
-      <link name="${prefix}finger_link_3">
+      <link name="${prefix}finger_r_link3">
          <visual>
             <origin xyz="0 0 0" rpy="0 0 0" />
@@ -136,7 +141,7 @@
          </inertial>
       </link>
-      <joint name="${prefix}finger_joint_4" type="revolute">
-         <parent link="${prefix}finger_link_3" />
-         <child link="${prefix}finger_link_4" />
+      <joint name="${prefix}finger_r_joint4" type="revolute">
+         <parent link="${prefix}finger_r_link3" />
+         <child link="${prefix}finger_r_link4" />
          <origin xyz="0.0 0.0 0.0355" rpy="0 0 0" />
          <axis xyz="0 1 0" />
@@ -144,5 +149,5 @@
          <dynamics damping="0.05" />
       </joint>
-      <link name="${prefix}finger_link_4">
+      <link name="${prefix}finger_r_link4">
          <visual>
             <origin xyz="0 0 0" rpy="0 0 0" />
@@ -171,10 +176,10 @@
          </inertial>
       </link>
-      <joint name="${prefix}finger_end_1" type="fixed">
-         <parent link="${prefix}finger_link_4" />
-         <child link="${prefix}finger_end_link_1" />
+      <joint name="${prefix}finger_end_r_joint1" type="fixed">
+         <parent link="${prefix}finger_r_link4" />
+         <child link="${prefix}finger_end_r_link1" />
          <origin xyz="0.0 0.0 0.02425" rpy="0 0 0" />
       </joint>
-      <link name="$(arg prefix)finger_end_link_1">
+      <link name="${prefix}finger_end_r_link1">
          <visual>
             <origin xyz="0 0 0" rpy="0 0 0"/>
@@ -188,7 +193,7 @@
       </link>
       <!-- INDEX -->
-      <joint name="${prefix}finger_joint_5" type="revolute">
-         <parent link="${prefix}robotis_hand_base" />
-         <child link="${prefix}finger_link_5" />
+      <joint name="${prefix}finger_r_joint5" type="revolute">
+         <parent link="${prefix}rh_5_right_base" />
+         <child link="${prefix}finger_r_link5" />
          <origin xyz="-0.002 0.03608 0.09575" rpy="0 0 0" />
          <axis xyz="1 0 0" />
@@ -196,5 +201,5 @@
          <dynamics damping="0.05" />
       </joint>
-      <link name="${prefix}finger_link_5">
+      <link name="${prefix}finger_r_link5">
          <visual>
             <origin xyz="0 0 0" rpy="0 0 0" />
@@ -223,7 +228,7 @@
          </inertial>
       </link>
-      <joint name="${prefix}finger_joint_6" type="revolute">
-         <parent link="${prefix}finger_link_5" />
-         <child link="${prefix}finger_link_6" />
+      <joint name="${prefix}finger_r_joint6" type="revolute">
+         <parent link="${prefix}finger_r_link5" />
+         <child link="${prefix}finger_r_link6" />
          <origin xyz="0.0165 0.0 0.0235" rpy="0 0 0" />
          <axis xyz="0 1 0" />
@@ -231,5 +236,5 @@
          <dynamics damping="0.05" />
       </joint>
-      <link name="${prefix}finger_link_6">
+      <link name="${prefix}finger_r_link6">
          <visual>
             <origin xyz="0 0 0" rpy="0 0 0" />
@@ -258,7 +263,7 @@
          </inertial>
       </link>
-      <joint name="${prefix}finger_joint_7" type="revolute">
-         <parent link="${prefix}finger_link_6" />
-         <child link="${prefix}finger_link_7" />
+      <joint name="${prefix}finger_r_joint7" type="revolute">
+         <parent link="${prefix}finger_r_link6" />
+         <child link="${prefix}finger_r_link7" />
          <origin xyz="0.0 0.0 0.0355" rpy="0 0 0" />
          <axis xyz="0 1 0" />
@@ -266,5 +271,5 @@
          <dynamics damping="0.05" />
       </joint>
-      <link name="${prefix}finger_link_7">
+      <link name="${prefix}finger_r_link7">
          <visual>
             <origin xyz="0 0 0" rpy="0 0 0" />
@@ -293,7 +298,7 @@
          </inertial>
       </link>
-      <joint name="${prefix}finger_joint_8" type="revolute">
-         <parent link="${prefix}finger_link_7" />
-         <child link="${prefix}finger_link_8" />
+      <joint name="${prefix}finger_r_joint8" type="revolute">
+         <parent link="${prefix}finger_r_link7" />
+         <child link="${prefix}finger_r_link8" />
          <origin xyz="0.0 0.0 0.0355" rpy="0 0 0" />
          <axis xyz="0 1 0" />
@@ -301,5 +306,5 @@
          <dynamics damping="0.05" />
       </joint>
-      <link name="${prefix}finger_link_8">
+      <link name="${prefix}finger_r_link8">
          <visual>
             <origin xyz="0 0 0" rpy="0 0 0" />
@@ -328,10 +333,10 @@
          </inertial>
       </link>
-      <joint name="${prefix}finger_end_2" type="fixed">
-         <parent link="${prefix}finger_link_8" />
-         <child link="${prefix}finger_end_link_2" />
+      <joint name="${prefix}finger_end_r_joint2" type="fixed">
+         <parent link="${prefix}finger_r_link8" />
+         <child link="${prefix}finger_end_r_link2" />
          <origin xyz="0.0 0.0 0.02425" rpy="0 0 0" />
       </joint>
-      <link name="$(arg prefix)finger_end_link_2">
+      <link name="${prefix}finger_end_r_link2">
          <visual>
             <origin xyz="0 0 0" rpy="0 0 0"/>
@@ -345,7 +350,7 @@
       </link>
       <!-- MIDDLE -->
-      <joint name="${prefix}finger_joint_9" type="revolute">
-         <parent link="${prefix}robotis_hand_base" />
-         <child link="${prefix}finger_link_9" />
+      <joint name="${prefix}finger_r_joint9" type="revolute">
+         <parent link="${prefix}rh_5_right_base" />
+         <child link="${prefix}finger_r_link9" />
          <origin xyz="-0.002 0.00908 0.10353" rpy="0 0 0" />
          <axis xyz="1 0 0" />
@@ -353,5 +358,5 @@
          <dynamics damping="0.05" />
       </joint>
-      <link name="${prefix}finger_link_9">
+      <link name="${prefix}finger_r_link9">
          <visual>
             <origin xyz="0 0 0" rpy="0 0 0" />
@@ -380,7 +385,7 @@
          </inertial>
       </link>
-      <joint name="${prefix}finger_joint_10" type="revolute">
-         <parent link="${prefix}finger_link_9" />
-         <child link="${prefix}finger_link_10" />
+      <joint name="${prefix}finger_r_joint10" type="revolute">
+         <parent link="${prefix}finger_r_link9" />
+         <child link="${prefix}finger_r_link10" />
          <origin xyz="0.0165 0.0 0.0235" rpy="0 0 0" />
          <axis xyz="0 1 0" />
@@ -388,5 +393,5 @@
          <dynamics damping="0.05" />
       </joint>
-      <link name="${prefix}finger_link_10">
+      <link name="${prefix}finger_r_link10">
          <visual>
             <origin xyz="0 0 0" rpy="0 0 0" />
@@ -415,7 +420,7 @@
          </inertial>
       </link>
-      <joint name="${prefix}finger_joint_11" type="revolute">
-         <parent link="${prefix}finger_link_10" />
-         <child link="${prefix}finger_link_11" />
+      <joint name="${prefix}finger_r_joint11" type="revolute">
+         <parent link="${prefix}finger_r_link10" />
+         <child link="${prefix}finger_r_link11" />
          <origin xyz="0.0 0.0 0.0355" rpy="0 0 0" />
          <axis xyz="0 1 0" />
@@ -423,5 +428,5 @@
          <dynamics damping="0.05" />
       </joint>
-      <link name="${prefix}finger_link_11">
+      <link name="${prefix}finger_r_link11">
          <visual>
             <origin xyz="0 0 0" rpy="0 0 0" />
@@ -450,7 +455,7 @@
          </inertial>
       </link>
-      <joint name="${prefix}finger_joint_12" type="revolute">
-         <parent link="${prefix}finger_link_11" />
-         <child link="${prefix}finger_link_12" />
+      <joint name="${prefix}finger_r_joint12" type="revolute">
+         <parent link="${prefix}finger_r_link11" />
+         <child link="${prefix}finger_r_link12" />
          <origin xyz="0.0 0.0 0.0355" rpy="0 0 0" />
          <axis xyz="0 1 0" />
@@ -458,5 +463,5 @@
          <dynamics damping="0.05" />
       </joint>
-      <link name="${prefix}finger_link_12">
+      <link name="${prefix}finger_r_link12">
          <visual>
             <origin xyz="0 0 0" rpy="0 0 0" />
@@ -485,10 +490,10 @@
          </inertial>
       </link>
-      <joint name="${prefix}finger_end_3" type="fixed">
-         <parent link="${prefix}finger_link_12" />
-         <child link="${prefix}finger_end_link_3" />
+      <joint name="${prefix}finger_end_r_joint3" type="fixed">
+         <parent link="${prefix}finger_r_link12" />
+         <child link="${prefix}finger_end_r_link3" />
          <origin xyz="0.0 0.0 0.02425" rpy="0 0 0" />
       </joint>
-      <link name="$(arg prefix)finger_end_link_3">
+      <link name="${prefix}finger_end_r_link3">
          <visual>
             <origin xyz="0 0 0" rpy="0 0 0"/>
@@ -502,7 +507,7 @@
       </link>
       <!-- RING -->
-      <joint name="${prefix}finger_joint_13" type="revolute">
-         <parent link="${prefix}robotis_hand_base" />
-         <child link="${prefix}finger_link_13" />
+      <joint name="${prefix}finger_r_joint13" type="revolute">
+         <parent link="${prefix}rh_5_right_base" />
+         <child link="${prefix}finger_r_link13" />
          <origin xyz="-0.002 -0.01792 0.09775" rpy="0 0 0" />
          <axis xyz="1 0 0" />
@@ -510,5 +515,5 @@
          <dynamics damping="0.05" />
       </joint>
-      <link name="${prefix}finger_link_13">
+      <link name="${prefix}finger_r_link13">
          <visual>
             <origin xyz="0 0 0" rpy="0 0 0" />
@@ -537,7 +542,7 @@
          </inertial>
       </link>
-      <joint name="${prefix}finger_joint_14" type="revolute">
-         <parent link="${prefix}finger_link_13" />
-         <child link="${prefix}finger_link_14" />
+      <joint name="${prefix}finger_r_joint14" type="revolute">
+         <parent link="${prefix}finger_r_link13" />
+         <child link="${prefix}finger_r_link14" />
          <origin xyz="0.0165 0.0 0.0235" rpy="0 0 0" />
          <axis xyz="0 1 0" />
@@ -545,5 +550,5 @@
          <dynamics damping="0.05" />
       </joint>
-      <link name="${prefix}finger_link_14">
+      <link name="${prefix}finger_r_link14">
          <visual>
             <origin xyz="0 0 0" rpy="0 0 0" />
@@ -572,7 +577,7 @@
          </inertial>
       </link>
-      <joint name="${prefix}finger_joint_15" type="revolute">
-         <parent link="${prefix}finger_link_14" />
-         <child link="${prefix}finger_link_15" />
+      <joint name="${prefix}finger_r_joint15" type="revolute">
+         <parent link="${prefix}finger_r_link14" />
+         <child link="${prefix}finger_r_link15" />
          <origin xyz="0.0 0.0 0.0355" rpy="0 0 0" />
          <axis xyz="0 1 0" />
@@ -580,5 +585,5 @@
          <dynamics damping="0.05" />
       </joint>
-      <link name="${prefix}finger_link_15">
+      <link name="${prefix}finger_r_link15">
          <visual>
             <origin xyz="0 0 0" rpy="0 0 0" />
@@ -607,7 +612,7 @@
          </inertial>
       </link>
-      <joint name="${prefix}finger_joint_16" type="revolute">
-         <parent link="${prefix}finger_link_15" />
-         <child link="${prefix}finger_link_16" />
+      <joint name="${prefix}finger_r_joint16" type="revolute">
+         <parent link="${prefix}finger_r_link15" />
+         <child link="${prefix}finger_r_link16" />
          <origin xyz="0.0 0.0 0.0355" rpy="0 0 0" />
          <axis xyz="0 1 0" />
@@ -615,5 +620,5 @@
          <dynamics damping="0.05" />
       </joint>
-      <link name="${prefix}finger_link_16">
+      <link name="${prefix}finger_r_link16">
          <visual>
             <origin xyz="0 0 0" rpy="0 0 0" />
@@ -642,10 +647,10 @@
          </inertial>
       </link>
-      <joint name="${prefix}finger_end_4" type="fixed">
-         <parent link="${prefix}finger_link_16" />
-         <child link="${prefix}finger_end_link_4" />
+      <joint name="${prefix}finger_end_r_joint4" type="fixed">
+         <parent link="${prefix}finger_r_link16" />
+         <child link="${prefix}finger_end_r_link4" />
          <origin xyz="0.0 0.0 0.02425" rpy="0 0 0" />
       </joint>
-      <link name="$(arg prefix)finger_end_link_4">
+      <link name="${prefix}finger_end_r_link4">
          <visual>
             <origin xyz="0 0 0" rpy="0 0 0"/>
@@ -659,7 +664,7 @@
       </link>
       <!-- PINKY -->
-      <joint name="${prefix}finger_joint_17" type="revolute">
-         <parent link="${prefix}robotis_hand_base" />
-         <child link="${prefix}finger_link_17" />
+      <joint name="${prefix}finger_r_joint17" type="revolute">
+         <parent link="${prefix}rh_5_right_base" />
+         <child link="${prefix}finger_r_link17" />
          <origin xyz="-0.002 -0.04492 0.07875" rpy="0 0 0" />
          <axis xyz="1 0 0" />
@@ -667,5 +672,5 @@
          <dynamics damping="0.05" />
       </joint>
-      <link name="${prefix}finger_link_17">
+      <link name="${prefix}finger_r_link17">
          <visual>
             <origin xyz="0 0 0" rpy="0 0 0" />
@@ -694,7 +699,7 @@
          </inertial>
       </link>
-      <joint name="${prefix}finger_joint_18" type="revolute">
-         <parent link="${prefix}finger_link_17" />
-         <child link="${prefix}finger_link_18" />
+      <joint name="${prefix}finger_r_joint18" type="revolute">
+         <parent link="${prefix}finger_r_link17" />
+         <child link="${prefix}finger_r_link18" />
          <origin xyz="0.0165 0.0 0.0235" rpy="0 0 0" />
          <axis xyz="0 1 0" />
@@ -702,5 +707,5 @@
          <dynamics damping="0.05" />
       </joint>
-      <link name="${prefix}finger_link_18">
+      <link name="${prefix}finger_r_link18">
          <visual>
             <origin xyz="0 0 0" rpy="0 0 0" />
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
Commit message: Added robotis_hand VR teleoperation packages. Updated URDF and meshes.
Signed-off-by: Hyunwoo Nam <nhw@robotis.com>

File: ffw_description/urdf/common/rh_5_left/rh_5_left.urdf.xacro (robot description, xacro)
@@ -196,5 +196,5 @@
          <parent link="${prefix}rh_5_left_base" />
          <child link="${prefix}finger_l_link5" />
-         <origin xyz="-0.002 -0.03608 0.09575" rpy="0 0 0" />
+         <origin xyz="-0.0015 -0.03608 0.09575" rpy="0 0 0" />
          <axis xyz="1 0 0" />
          <limit velocity="4.8" effort="1000" lower="-0.6" upper="0.6" />
@@ -353,5 +353,5 @@
          <parent link="${prefix}rh_5_left_base" />
          <child link="${prefix}finger_l_link9" />
-         <origin xyz="-0.002 -0.00908 0.10353" rpy="0 0 0" />
+         <origin xyz="-0.0015 -0.00908 0.10353" rpy="0 0 0" />
          <axis xyz="1 0 0" />
          <limit velocity="4.8" effort="1000" lower="-0.6" upper="0.6" />
@@ -510,5 +510,5 @@
          <parent link="${prefix}rh_5_left_base" />
          <child link="${prefix}finger_l_link13" />
-         <origin xyz="-0.002 0.01792 0.09775" rpy="0 0 0" />
+         <origin xyz="-0.0015 0.01792 0.09775" rpy="0 0 0" />
          <axis xyz="1 0 0" />
          <limit velocity="4.8" effort="1000" lower="-0.6" upper="0.6" />
@@ -667,5 +667,5 @@
          <parent link="${prefix}rh_5_left_base" />
          <child link="${prefix}finger_l_link17" />
-         <origin xyz="-0.002 0.04492 0.07875" rpy="0 0 0" />
+         <origin xyz="-0.0015 0.04492 0.07875" rpy="0 0 0" />
          <axis xyz="1 0 0" />
          <limit velocity="4.8" effort="1000" lower="-0.6" upper="0.6" />

File: ffw_description/urdf/common/rh_5_right/rh_5_right.urdf.xacro (robot description, xacro)
@@ -28,9 +28,9 @@
          </collision>
          <inertial>
-            <origin xyz="-1.033899300e-03 2.272987300e-03 6.124897700e-02" />
-            <mass value="2.823506000e-01" />
-            <inertia ixx="4.620917800e-04" ixy="-2.064753200e-06" ixz="5.785037100e-06"
-            iyy="2.969158600e-04" iyz="-2.128225400e-05"
-            izz="2.153594900e-04" />
+            <origin xyz="-1.6731925e-03 1.2908873e-03 6.0855215e-02" />
+            <mass value="3.5306225e-01" />
+            <inertia ixx="5.9371826e-04" ixy="-1.9267347e-06" ixz="-4.6360975e-06"
+            iyy="3.8516622e-04" iyz="-2.0206128e-05"
+            izz="3.1560646e-04" />
          </inertial>
       </link>
@@ -196,5 +196,5 @@
          <parent link="${prefix}rh_5_right_base" />
          <child link="${prefix}finger_r_link5" />
-         <origin xyz="-0.002 0.03608 0.09575" rpy="0 0 0" />
+         <origin xyz="-0.0015 0.03608 0.09575" rpy="0 0 0" />
          <axis xyz="1 0 0" />
          <limit velocity="4.8" effort="1000" lower="-0.6" upper="0.6" />
@@ -353,5 +353,5 @@
          <parent link="${prefix}rh_5_right_base" />
          <child link="${prefix}finger_r_link9" />
-         <origin xyz="-0.002 0.00908 0.10353" rpy="0 0 0" />
+         <origin xyz="-0.0015 0.00908 0.10353" rpy="0 0 0" />
          <axis xyz="1 0 0" />
          <limit velocity="4.8" effort="1000" lower="-0.6" upper="0.6" />
@@ -510,5 +510,5 @@
          <parent link="${prefix}rh_5_right_base" />
          <child link="${prefix}finger_r_link13" />
-         <origin xyz="-0.002 -0.01792 0.09775" rpy="0 0 0" />
+         <origin xyz="-0.0015 -0.01792 0.09775" rpy="0 0 0" />
          <axis xyz="1 0 0" />
          <limit velocity="4.8" effort="1000" lower="-0.6" upper="0.6" />
@@ -667,5 +667,5 @@
          <parent link="${prefix}rh_5_right_base" />
          <child link="${prefix}finger_r_link17" />
-         <origin xyz="-0.002 -0.04492 0.07875" rpy="0 0 0" />
+         <origin xyz="-0.0015 -0.04492 0.07875" rpy="0 0 0" />
          <axis xyz="1 0 0" />
          <limit velocity="4.8" effort="1000" lower="-0.6" upper="0.6" />
