Commit message: feat: Add IMU joint and link to URDF for improved sensor integration

File: ffw_description/urdf/ffw_sg2_rev1_follower/ffw_sg2_follower.urdf.xacro (robot description, xacro)
@@ -50,4 +50,11 @@
   </joint>
   <link name="$(arg prefix)lidar_r_link">
+  </link>
+  <joint name="$(arg prefix)imu_joint" type="fixed">
+    <parent link="$(arg prefix)base_link"/>
+    <child link="$(arg prefix)imu_link"/>
+    <origin xyz="-0.1464 0.0 0.26" rpy="0 0 0"/>
+  </joint>
+  <link name="$(arg prefix)imu_link">
   </link>
   <link name="$(arg prefix)lift_link">

Commit message: fix: Adjust Lidar joint orientations in URDF for correct alignment

File: ffw_description/urdf/ffw_sg2_rev1_follower/ffw_sg2_follower.urdf.xacro (robot description, xacro)
@@ -40,5 +40,5 @@
     <parent link="$(arg prefix)base_link"/>
     <child link="$(arg prefix)lidar_l_link"/>
-    <origin xyz="-0.111881 0.240 0.34432" rpy="0 0 0"/>
+    <origin xyz="-0.111881 0.240 0.34432" rpy="0 0 1.57079632679"/>
   </joint>
   <link name="$(arg prefix)lidar_l_link">
@@ -47,5 +47,5 @@
     <parent link="$(arg prefix)base_link"/>
     <child link="$(arg prefix)lidar_r_link"/>
-    <origin xyz="-0.111881 -0.240 0.34432" rpy="0 0 0"/>
+    <origin xyz="-0.111881 -0.240 0.34432" rpy="0 0 -1.57079632679"/>
   </joint>
   <link name="$(arg prefix)lidar_r_link">
