Commit message: Modified urdfs, vr publisher

File: ffw_description/urdf/ffw_sg2_rev1_follower/ffw_sg2_follower.urdf (robot description, URDF)
Before this commit: robot ffw_sg2_follower, 40 links, 39 joints
Links:
- added link end_effector_l_link; visual box size=0.01 0.01 0.01
- added link end_effector_r_link; visual box size=0.01 0.01 0.01
- link arm_base_link: geometry collision box size=0.2 0.1 0.63; collision box size=0.2 0.1 0.63
- link arm_l_link1: geometry visual mesh filename=package://ffw_description/meshes/common/follower/arm_l_link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 scale=0.001 0.001 0.001
- link arm_l_link2: geometry collision cylinder length=0.30 radius=0.07; collision sphere radius=0.07
- link arm_l_link3: geometry visual mesh filename=package://ffw_description/meshes/common/follower/arm_l_link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 scale=0.001 0.001 0.001
- link arm_l_link4: geometry collision cylinder length=0.3 radius=0.07; collision sphere radius=0.07
- link arm_l_link5: geometry visual mesh filename=package://ffw_description/meshes/common/follower/arm_l_link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 scale=0.001 0.001 0.001
- link arm_l_link6: geometry visual mesh filename=package://ffw_description/meshes/common/follower/arm_l_link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 scale=0.001 0.001 0.001
- link arm_l_link7: geometry collision cylinder length=0.12 radius=0.085; collision sphere radius=0.085
- link arm_r_link1: geometry visual mesh filename=package://ffw_description/meshes/common/follower/arm_r_link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 scale=0.001 0.001 0.001
- link arm_r_link2: geometry collision cylinder length=0.30 radius=0.07; collision sphere radius=0.07
- link arm_r_link3: geometry visual mesh filename=package://ffw_description/meshes/common/follower/arm_r_link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 scale=0.001 0.001 0.001
- link arm_r_link4: geometry collision cylinder length=0.3 radius=0.07; collision sphere radius=0.07
- link arm_r_link5: geometry visual mesh filename=package://ffw_description/meshes/common/follower/arm_r_link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 scale=0.001 0.001 0.001
- link arm_r_link6: geometry visual mesh filename=package://ffw_description/meshes/common/follower/arm_r_link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 scale=0.001 0.001 0.001
- link arm_r_link7: geometry collision cylinder length=0.12 radius=0.085; collision sphere radius=0.085
- link base_link: mass 3.598943900e+01 -> 35.989; geometry visual mesh filename=package://ffw_description/meshes/ffw_sg2_rev1_follower/base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 scale=0.001 0.001 0.001
- link camera_l_link: geometry visual mesh filename=file:///root/ros2_ws/install/realsense2_description/share/r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 scale=0.001 0.001 0.001
- link camera_r_link: geometry visual mesh filename=file:///root/ros2_ws/install/realsense2_description/share/r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 scale=0.001 0.001 0.001
- link gripper_l_rh_p12_rn_base: geometry visual mesh filename=package://ffw_description/meshes/common/rh_p12_rn_a/base.stl scale=0.001 0.001 0.001
- link gripper_l_rh_p12_rn_l1: geometry visual mesh filename=package://ffw_description/meshes/common/rh_p12_rn_a/l1.stl scale=0.001 0.001 0.001
- link gripper_l_rh_p12_rn_l2: geometry visual mesh filename=package://ffw_description/meshes/common/rh_p12_rn_a/l2.stl scale=0.001 0.001 0.001
- link gripper_l_rh_p12_rn_r1: geometry visual mesh filename=package://ffw_description/meshes/common/rh_p12_rn_a/r1.stl scale=0.001 0.001 0.001
- link gripper_l_rh_p12_rn_r2: geometry visual mesh filename=package://ffw_description/meshes/common/rh_p12_rn_a/r2.stl scale=0.001 0.001 0.001
- link gripper_r_rh_p12_rn_base: geometry visual mesh filename=package://ffw_description/meshes/common/rh_p12_rn_a/base.stl scale=0.001 0.001 0.001
- link gripper_r_rh_p12_rn_l1: geometry visual mesh filename=package://ffw_description/meshes/common/rh_p12_rn_a/l1.stl scale=0.001 0.001 0.001
- link gripper_r_rh_p12_rn_l2: geometry visual mesh filename=package://ffw_description/meshes/common/rh_p12_rn_a/l2.stl scale=0.001 0.001 0.001
- link gripper_r_rh_p12_rn_r1: geometry visual mesh filename=package://ffw_description/meshes/common/rh_p12_rn_a/r1.stl scale=0.001 0.001 0.001
- link gripper_r_rh_p12_rn_r2: geometry visual mesh filename=package://ffw_description/meshes/common/rh_p12_rn_a/r2.stl scale=0.001 0.001 0.001
- link head_link1: geometry visual mesh filename=package://ffw_description/meshes/common/follower/head_link1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 scale=0.001 0.001 0.001
- link head_link2: geometry collision sphere radius=0.1; visual mesh filename=package://ffw_description/meshes/common/follower/head_link2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 scale=0.001 0.001 0.001
- link left_wheel_drive_link: geometry visual mesh filename=package://ffw_description/meshes/ffw_sg2_rev1_follower/left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 scale=0.001 0.001 0.001
- link left_wheel_steer_link: geometry visual mesh filename=package://ffw_description/meshes/ffw_sg2_rev1_follower/left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 scale=0.001 0.001 0.001
- link lift_link: mass 1.790000000e+01 -> 17.9; geometry visual mesh filename=package://ffw_description/meshes/ffw_sg2_rev1_follower/lift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 scale=0.001 0.001 0.001
- link rear_wheel_drive_link: geometry visual mesh filename=package://ffw_description/meshes/ffw_sg2_rev1_follower/rear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 scale=0.001 0.001 0.001
- link rear_wheel_steer_link: geometry visual mesh filename=package://ffw_description/meshes/ffw_sg2_rev1_follower/rear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 scale=0.001 0.001 0.001
- link right_wheel_drive_link: geometry visual mesh filename=package://ffw_description/meshes/ffw_sg2_rev1_follower/righ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 scale=0.001 0.001 0.001
- link right_wheel_steer_link: geometry visual mesh filename=package://ffw_description/meshes/ffw_sg2_rev1_follower/righ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 scale=0.001 0.001 0.001
Joints:
- added joint end_effector_l_joint: type fixed, parent arm_l_link7, child end_effector_l_link, origin xyz=0 0 -0.215 rpy=0 0 0
- added joint end_effector_r_joint: type fixed, parent arm_r_link7, child end_effector_r_link, origin xyz=0 0 -0.215 rpy=0 0 0
- joint arm_l_joint1: limit lower=-3.14 upper=3.14 effort=1000 velocity=4.8 -> lower=-3.14 upper=1.5707 effort=1000 velocity=4.8
- joint arm_l_joint4: limit lower=-2.9361 upper=1.0786 effort=1000 velocity=4.8 -> lower=-2.9361 upper=-0.7 effort=1000 velocity=4.8
- joint arm_r_joint1: limit lower=-3.14 upper=3.14 effort=1000 velocity=4.8 -> lower=-3.14 upper=1.5707 effort=1000 velocity=4.8
- joint arm_r_joint4: limit lower=-2.9361 upper=1.0786 effort=1000 velocity=4.8 -> lower=-2.9361 upper=-0.7 effort=1000 velocity=4.8
- joint gripper_l_joint1: type revolute -> fixed
- joint gripper_l_joint2: type revolute -> fixed
- joint gripper_l_joint3: type revolute -> fixed
- joint gripper_l_joint4: type revolute -> fixed
- joint gripper_r_joint1: type revolute -> fixed
- joint gripper_r_joint2: type revolute -> fixed
- joint gripper_r_joint3: type revolute -> fixed
- joint gripper_r_joint4: type revolute -> fixed
- joint head_joint1: type revolute -> fixed
- joint head_joint2: type revolute -> fixed
- joint left_wheel_drive: type revolute -> fixed
- joint left_wheel_steer: type revolute -> fixed
- joint lift_joint: type prismatic -> fixed
- joint rear_wheel_drive: type revolute -> fixed
- joint rear_wheel_steer: type revolute -> fixed
- joint right_wheel_drive: type revolute -> fixed
- joint right_wheel_steer: type revolute -> fixed
