Commit message: Added dummy gripper joints to bh5
Signed-off-by: Hyunwoo Nam <nhw@robotis.com>

File: ffw_description/urdf/ffw_bh5_rev1_follower/ffw_bh5_follower.urdf.xacro (robot description, xacro)
@@ -55,4 +55,36 @@
     use_fake_hardware="$(arg use_fake_hardware)"
     fake_sensor_commands="$(arg fake_sensor_commands)"/>
+  <joint name="$(arg prefix)gripper_r_joint1" type="revolute">
+      <parent link="$(arg prefix)base_link" />
+      <child link="$(arg prefix)dummy_link1" />
+      <origin xyz="0.0 0.0 0.0" rpy="0 0 0" />
+  </joint>
+  <link name="$(arg prefix)dummy_link1">
+      <visual>
+        <origin xyz="0 0 0" rpy="0 0 0"/>
+        <geometry>
+        <box size="0.01 0.01 0.01" />
+        </geometry>
+        <material name="red">
+        <color rgba="1.0 0.0 0.0 1"/>
+        </material>
+      </visual>
+  </link>
+  <joint name="$(arg prefix)gripper_l_joint1" type="revolute">
+      <parent link="$(arg prefix)base_link" />
+      <child link="$(arg prefix)dummy_link2" />
+      <origin xyz="0.0 0.0 0.0" rpy="0 0 0" />
+  </joint>
+  <link name="$(arg prefix)dummy_link2">
+      <visual>
+        <origin xyz="0 0 0" rpy="0 0 0"/>
+        <geometry>
+        <box size="0.01 0.01 0.01" />
+        </geometry>
+        <material name="red">
+        <color rgba="1.0 0.0 0.0 1"/>
+        </material>
+      </visual>
+  </link>
   <gazebo>
       <plugin filename="gz_ros2_control-system" name="gz_ros2_control::GazeboSimROS2ControlPlugin">
