Commit message: Updated ros2 control xacro files

File: ffw_description/ros2_control/ffw_bg2_rev4_follower/ffw_bg2_follower.ros2_control.xacro (robot description, xacro)
@@ -23,8 +23,8 @@
             <param name="number_of_transmissions">19</param>
             <param name="disable_torque_at_init">true</param>
-            <param name="dynamixel_state_pub_msg_name">dynamixel_hardware_interface/dxl_state</param>
-            <param name="get_dynamixel_data_srv_name">dynamixel_hardware_interface/get_dxl_data</param>
-            <param name="set_dynamixel_data_srv_name">dynamixel_hardware_interface/set_dxl_data</param>
-            <param name="reboot_dxl_srv_name">dynamixel_hardware_interface/reboot_dxl</param>
+            <param name="dynamixel_state_pub_msg_name">ffw_follower/dxl_state</param>
+            <param name="get_dynamixel_data_srv_name">ffw_follower/get_dxl_data</param>
+            <param name="set_dynamixel_data_srv_name">ffw_follower/set_dxl_data</param>
+            <param name="reboot_dxl_srv_name">ffw_follower/reboot_dxl</param>
             <param name="set_dxl_torque_srv_name">dynamixel_hardware_interface/set_dxl_torque</param>
           </xacro:unless>

File: ffw_description/ros2_control/ffw_bh5_rev1_follower/ffw_bh5_follower.ros2_control.xacro (robot description, xacro)
@@ -20,6 +20,6 @@
             <param name="baud_rate">4000000</param>
             <param name="dynamixel_model_folder">/param/dxl_model</param>
-            <param name="number_of_joints">59</param>
-            <param name="number_of_transmissions">59</param>
+            <param name="number_of_joints">57</param>
+            <param name="number_of_transmissions">57</param>
             <param name="disable_torque_at_init">true</param>
             <param name="dynamixel_state_pub_msg_name">dynamixel_hardware_interface/dxl_state</param>
@@ -686,5 +686,5 @@
         <param name="Startup Configuration">2</param>
         <param name="Operating Mode">5</param>
-        <param name="Drive Mode">13</param>
+        <param name="Drive Mode">12</param>
         <param name="Bus Watchdog">100</param>
         <param name="Profile Velocity">100</param>
@@ -710,5 +710,5 @@
         <param name="Startup Configuration">2</param>
         <param name="Operating Mode">5</param>
-        <param name="Drive Mode">13</param>
+        <param name="Drive Mode">12</param>
         <param name="Bus Watchdog">100</param>
         <param name="Profile Velocity">100</param>
@@ -733,5 +733,5 @@
         <param name="Startup Configuration">2</param>
         <param name="Operating Mode">5</param>
-        <param name="Drive Mode">13</param>
+        <param name="Drive Mode">12</param>
         <param name="Bus Watchdog">100</param>
         <param name="Profile Velocity">100</param>
@@ -1588,17 +1588,4 @@
         <param name="Max Position Limit">131875</param>
         <param name="Min Position Limit">-151875</param>
-      </gpio>
-      <gpio name="dxl8">
-        <param name="type">dxl</param>
-        <param name="ID">8</param>
-        <command_interface name="Goal Position"/>
-        <state_interface name="Present Position"/>
-        <state_interface name="Present Velocity"/>
-        <state_interface name="Present Current"/>
-        <state_interface name="Hardware Error Status"/>
-        <param name="Operating Mode">5</param>
-        <param name="Return Delay Time">0</param>
-        <param name="Profile Velocity">0</param>
-        <param name="Profile Acceleration">0</param>
       </gpio>
       <!-- LEFT HAND -->
@@ -1741,5 +1728,5 @@
         <param name="Startup Configuration">2</param>
         <param name="Operating Mode">5</param>
-        <param name="Drive Mode">12</param>
+        <param name="Drive Mode">13</param>
         <param name="Bus Watchdog">100</param>
         <param name="Profile Velocity">100</param>
@@ -1789,5 +1776,5 @@
         <param name="Startup Configuration">2</param>
         <param name="Operating Mode">5</param>
-        <param name="Drive Mode">12</param>
+        <param name="Drive Mode">13</param>
         <param name="Bus Watchdog">100</param>
         <param name="Profile Velocity">100</param>
@@ -1812,5 +1799,5 @@
         <param name="Startup Configuration">2</param>
         <param name="Operating Mode">5</param>
-        <param name="Drive Mode">12</param>
+        <param name="Drive Mode">13</param>
         <param name="Bus Watchdog">100</param>
         <param name="Profile Velocity">100</param>
@@ -2667,17 +2654,4 @@
         <param name="Max Position Limit">131875</param>
         <param name="Min Position Limit">-151875</param>
-      </gpio>
-      <gpio name="dxl38">
-        <param name="type">dxl</param>
-        <param name="ID">38</param>
-        <command_interface name="Goal Position"/>
-        <state_interface name="Present Position"/>
-        <state_interface name="Present Velocity"/>
-        <state_interface name="Present Current"/>
-        <state_interface name="Hardware Error Status"/>
-        <param name="Operating Mode">5</param>
-        <param name="Return Delay Time">0</param>
-        <param name="Profile Velocity">0</param>
-        <param name="Profile Acceleration">0</param>
       </gpio>
       <!-- LIFT -->
@@ -2748,9 +2722,9 @@
         <param name="Max Position Limit">2275</param>
         <param name="Min Position Limit">1820</param>
-        <param name="Position P Gain">1600</param>
-        <param name="Position I Gain">400</param>
-        <param name="Position D Gain">400</param>
-        <param name="Feedforward 1st Gain">30</param>
-        <param name="Feedforward 2nd Gain">30</param>
+        <param name="Position P Gain">800</param>
+        <param name="Position I Gain">200</param>
+        <param name="Position D Gain">200</param>
+        <param name="Feedforward 1st Gain">20</param>
+        <param name="Feedforward 2nd Gain">20</param>
       </gpio>
     </ros2_control>

File: ffw_description/ros2_control/ffw_sg2_rev1_follower/ffw_sg2_follower.ros2_control.xacro (robot description, xacro)
@@ -586,9 +586,9 @@
         <param name="Max Position Limit">2275</param>
         <param name="Min Position Limit">1820</param>
-        <param name="Position P Gain">1600</param>
-        <param name="Position I Gain">400</param>
-        <param name="Position D Gain">400</param>
-        <param name="Feedforward 1st Gain">30</param>
-        <param name="Feedforward 2nd Gain">30</param>
+        <param name="Position P Gain">800</param>
+        <param name="Position I Gain">200</param>
+        <param name="Position D Gain">200</param>
+        <param name="Feedforward 1st Gain">20</param>
+        <param name="Feedforward 2nd Gain">20</param>
       </gpio>
       <!-- LEFT WHEEL -->

File: ffw_description/ros2_control/ffw_sh5_rev1_follower/ffw_sh5_follower.ros2_control.xacro (robot description, xacro)
@@ -1,6 +1,6 @@
 <?xml version="1.0"?>
 <robot xmlns:xacro="http://www.ros.org/wiki/xacro">
-  <xacro:macro name="ffw_sh5_follower_system" params="use_sim:=^|false use_mock_hardware:=^|false mock_sensor_commands:=^|false">
-    <ros2_control name="ffw_sh5_follower" type="system" is_async="true">
+  <xacro:macro name="ffw_sg2_follower_system" params="use_sim:=^|false use_mock_hardware:=^|false mock_sensor_commands:=^|false">
+    <ros2_control name="ffw_sg2_follower" type="system" is_async="true">
       <xacro:if value="$(arg use_sim)">
         <hardware>
@@ -11,5 +11,5 @@
         <hardware>
           <xacro:if value="${use_mock_hardware}">
-            <plugin>fake_components/GenericSystem</plugin>
+            <plugin>mock_components/GenericSystem</plugin>
             <param name="mock_sensor_commands">${mock_sensor_commands}</param>
             <param name="state_following_offset">0.0</param>
@@ -23,8 +23,8 @@
             <param name="number_of_transmissions">60</param>
             <param name="disable_torque_at_init">true</param>
-            <param name="dynamixel_state_pub_msg_name">dynamixel_hardware_interface/dxl_state</param>
-            <param name="get_dynamixel_data_srv_name">dynamixel_hardware_interface/get_dxl_data</param>
-            <param name="set_dynamixel_data_srv_name">dynamixel_hardware_interface/set_dxl_data</param>
-            <param name="reboot_dxl_srv_name">dynamixel_hardware_interface/reboot_dxl</param>
+            <param name="dynamixel_state_pub_msg_name">ffw_follower/dxl_state</param>
+            <param name="get_dynamixel_data_srv_name">ffw_follower/get_dxl_data</param>
+            <param name="set_dynamixel_data_srv_name">ffw_follower/set_dxl_data</param>
+            <param name="reboot_dxl_srv_name">ffw_follower/reboot_dxl</param>
             <param name="set_dxl_torque_srv_name">dynamixel_hardware_interface/set_dxl_torque</param>
           </xacro:unless>
@@ -704,5 +704,5 @@
         <param name="Startup Configuration">2</param>
         <param name="Operating Mode">5</param>
-        <param name="Drive Mode">13</param>
+        <param name="Drive Mode">12</param>
         <param name="Bus Watchdog">100</param>
         <param name="Profile Velocity">100</param>
@@ -728,5 +728,5 @@
         <param name="Startup Configuration">2</param>
         <param name="Operating Mode">5</param>
-        <param name="Drive Mode">13</param>
+        <param name="Drive Mode">12</param>
         <param name="Bus Watchdog">100</param>
         <param name="Profile Velocity">100</param>
@@ -751,5 +751,5 @@
         <param name="Startup Configuration">2</param>
         <param name="Operating Mode">5</param>
-        <param name="Drive Mode">13</param>
+        <param name="Drive Mode">12</param>
         <param name="Bus Watchdog">100</param>
         <param name="Profile Velocity">100</param>
@@ -1452,4 +1452,5 @@
         <state_interface name="Present Current"/>
         <state_interface name="Error Code"/>
+        <state_interface name="Present Input Voltage"/>
         <param name="Drive Mode">69</param>
         <param name="Operating Mode">3</param>
@@ -1457,4 +1458,6 @@
         <param name="Velocity Limit">3591</param>
         <param name="Acceleration Limit">35910</param>
+        <param name="Profile Velocity">3591</param>
+        <param name="Profile Acceleration">3591</param>
         <param name="Profile Acceleration Time">250</param>
         <param name="Profile Time">500</param>
@@ -1479,4 +1482,6 @@
         <param name="Velocity Limit">3591</param>
         <param name="Acceleration Limit">35910</param>
+        <param name="Profile Velocity">3591</param>
+        <param name="Profile Acceleration">3591</param>
         <param name="Profile Acceleration Time">250</param>
         <param name="Profile Time">500</param>
@@ -1501,4 +1506,6 @@
         <param name="Velocity Limit">3591</param>
         <param name="Acceleration Limit">35910</param>
+        <param name="Profile Velocity">3591</param>
+        <param name="Profile Acceleration">3591</param>
         <param name="Profile Acceleration Time">250</param>
         <param name="Profile Time">500</param>
@@ -1523,4 +1530,6 @@
         <param name="Velocity Limit">6486</param>
         <param name="Acceleration Limit">35910</param>
+        <param name="Profile Velocity">6486</param>
+        <param name="Profile Acceleration">3591</param>
         <param name="Profile Acceleration Time">250</param>
         <param name="Profile Time">500</param>
@@ -1545,4 +1554,6 @@
         <param name="Velocity Limit">6486</param>
         <param name="Acceleration Limit">35910</param>
+        <param name="Profile Velocity">6486</param>
+        <param name="Profile Acceleration">3591</param>
         <param name="Profile Acceleration Time">250</param>
         <param name="Profile Time">500</param>
@@ -1567,4 +1578,6 @@
         <param name="Velocity Limit">6486</param>
         <param name="Acceleration Limit">35910</param>
+        <param name="Profile Velocity">6486</param>
+        <param name="Profile Acceleration">3591</param>
         <param name="Profile Acceleration Time">250</param>
         <param name="Profile Time">500</param>
@@ -1589,5 +1602,5 @@
         <param name="Velocity Limit">2920</param>
         <param name="Acceleration Limit">359100</param>
-        <param name="Current Limit">1000</param>
+        <param name="Current Limit">1500</param>
         <param name="Profile Velocity">100</param>
         <param name="Profile Acceleration">50</param>
@@ -1734,5 +1747,5 @@
         <param name="Startup Configuration">2</param>
         <param name="Operating Mode">5</param>
-        <param name="Drive Mode">12</param>
+        <param name="Drive Mode">13</param>
         <param name="Bus Watchdog">100</param>
         <param name="Profile Velocity">100</param>
@@ -1782,5 +1795,5 @@
         <param name="Startup Configuration">2</param>
         <param name="Operating Mode">5</param>
-        <param name="Drive Mode">12</param>
+        <param name="Drive Mode">13</param>
         <param name="Bus Watchdog">100</param>
         <param name="Profile Velocity">100</param>
@@ -1805,5 +1818,5 @@
         <param name="Startup Configuration">2</param>
         <param name="Operating Mode">5</param>
-        <param name="Drive Mode">12</param>
+        <param name="Drive Mode">13</param>
         <param name="Bus Watchdog">100</param>
         <param name="Profile Velocity">100</param>
@@ -2511,4 +2524,6 @@
         <param name="Velocity Limit">3591</param>
         <param name="Acceleration Limit">35910</param>
+        <param name="Profile Velocity">3591</param>
+        <param name="Profile Acceleration">3591</param>
         <param name="Profile Acceleration Time">250</param>
         <param name="Profile Time">500</param>
@@ -2533,4 +2548,6 @@
         <param name="Velocity Limit">3591</param>
         <param name="Acceleration Limit">35910</param>
+        <param name="Profile Velocity">3591</param>
+        <param name="Profile Acceleration">3591</param>
         <param name="Profile Acceleration Time">250</param>
         <param name="Profile Time">500</param>
@@ -2555,4 +2572,6 @@
         <param name="Velocity Limit">3591</param>
         <param name="Acceleration Limit">35910</param>
+        <param name="Profile Velocity">3591</param>
+        <param name="Profile Acceleration">3591</param>
         <param name="Profile Acceleration Time">250</param>
         <param name="Profile Time">500</param>
@@ -2577,4 +2596,6 @@
         <param name="Velocity Limit">6486</param>
         <param name="Acceleration Limit">35910</param>
+        <param name="Profile Velocity">6486</param>
+        <param name="Profile Acceleration">3591</param>
         <param name="Profile Acceleration Time">250</param>
         <param name="Profile Time">500</param>
@@ -2599,4 +2620,6 @@
         <param name="Velocity Limit">6486</param>
         <param name="Acceleration Limit">35910</param>
+        <param name="Profile Velocity">6486</param>
+        <param name="Profile Acceleration">3591</param>
         <param name="Profile Acceleration Time">250</param>
         <param name="Profile Time">500</param>
@@ -2621,4 +2644,6 @@
         <param name="Velocity Limit">6486</param>
         <param name="Acceleration Limit">35910</param>
+        <param name="Profile Velocity">6486</param>
+        <param name="Profile Acceleration">3591</param>
         <param name="Profile Acceleration Time">250</param>
         <param name="Profile Time">500</param>
@@ -2643,5 +2668,5 @@
         <param name="Velocity Limit">2920</param>
         <param name="Acceleration Limit">359100</param>
-        <param name="Current Limit">1000</param>
+        <param name="Current Limit">1500</param>
         <param name="Profile Velocity">100</param>
         <param name="Profile Acceleration">50</param>
@@ -2672,9 +2697,15 @@
         <param name="Velocity P Gain">41387</param>
         <param name="Velocity I Gain">1065630</param>
+        <param name="[unit info]">
+          Present Position,0.00001,m,signed,0.0;
+          Goal Position,0.00001,m,signed,0.0;
+          Present Velocity,0.00087381333,m/s,signed,0.0;
+          Goal Velocity,0.00087381333,m/s,signed,0.0;
+        </param>
       </gpio>
       <!-- HEAD -->
       <gpio name="dxl61">
         <param name="type">dxl</param>
-        <param name="ID">61</param>z
+        <param name="ID">61</param>
         <command_interface name="Goal Position"/>
         <state_interface name="Present Position"/>
@@ -2682,5 +2713,6 @@
         <state_interface name="Present Current"/>
         <state_interface name="Hardware Error Status"/>
-        <param name="Drive Mode">1</param>
+        <state_interface name="Present Input Voltage"/>
+        <param name="Drive Mode">5</param>
         <param name="Operating Mode">3</param>
         <param name="Return Delay Time">0</param>
@@ -2703,5 +2735,5 @@
         <state_interface name="Present Current"/>
         <state_interface name="Hardware Error Status"/>
-        <param name="Drive Mode">1</param>
+        <param name="Drive Mode">5</param>
         <param name="Operating Mode">3</param>
         <param name="Return Delay Time">0</param>
@@ -2713,6 +2745,6 @@
         <param name="Position I Gain">200</param>
         <param name="Position D Gain">200</param>
-        <param name="Feedforward 1st Gain">30</param>
-        <param name="Feedforward 2nd Gain">30</param>
+        <param name="Feedforward 1st Gain">20</param>
+        <param name="Feedforward 2nd Gain">20</param>
       </gpio>
       <!-- LEFT WHEEL -->
