Commit message: modified gazebo nav2

File: ffw_description/gazebo/ffw_sg2_rev1_follower/ffw_sg2_follower.gazebo.xacro (robot description, xacro)
@@ -1,5 +1,6 @@
 <?xml version="1.0"?>
 <robot xmlns:xacro="http://ros.org/wiki/xacro">
-  <xacro:macro name="ffw_sg2_follower_gazebo" >
+  <!-- prefix is optional; default empty for non-prefixed TF/frames -->
+  <xacro:macro name="ffw_sg2_follower_gazebo" params="prefix:=">
   <xacro:macro name="SimpleTransmission" params="trans joint actuator">
     <transmission name="${trans}">
@@ -77,4 +78,65 @@
   <xacro:SimpleTransmission trans="l_tran_l1" joint="l_rh_l1" actuator="l_actuator3" />
   <xacro:SimpleTransmission trans="l_tran_l2" joint="l_rh_l2" actuator="l_actuator4" />
+  <!-- GZ lidar sensors for simulation (publish Gazebo LaserScan; bridge to ROS if needed) -->
+  <gazebo reference="lidar_l_link">
+    <sensor name="lidar_left" type="gpu_lidar">
+      <pose>-0 0 0 0 0 0</pose>
+      <always_on>true</always_on>
+      <visualize>true</visualize>
+      <update_rate>10.0</update_rate>
+      <ray>
+        <scan>
+          <horizontal>
+            <samples>720</samples>
+            <resolution>1</resolution>
+            <min_angle>-2.356194</min_angle>
+            <max_angle>2.356194</max_angle>
+          </horizontal>
+        </scan>
+        <range>
+          <min>0.05</min>
+          <max>20.0</max>
+          <resolution>0.01</resolution>
+        </range>
+        <noise>
+          <type>gaussian</type>
+          <mean>0.0</mean>
+          <stddev>0.01</stddev>
+        </noise>
+      </ray>
+      <gz_frame_id>lidar_l_link</gz_frame_id>
+      <topic>scan_left</topic>
+    </sensor>
+  </gazebo>
+  <gazebo reference="lidar_r_link">
+    <sensor name="lidar_right" type="gpu_lidar">
+      <pose>0 0 0 0 0 0</pose>
+      <always_on>true</always_on>
+      <visualize>true</visualize>
+      <update_rate>10.0</update_rate>
+      <ray>
+        <scan>
+          <horizontal>
+            <samples>720</samples>
+            <resolution>1</resolution>
+            <min_angle>-2.356194</min_angle>
+            <max_angle>2.356194</max_angle>
+          </horizontal>
+        </scan>
+        <range>
+          <min>0.05</min>
+          <max>20.0</max>
+          <resolution>0.01</resolution>
+        </range>
+        <noise>
+          <type>gaussian</type>
+          <mean>0.0</mean>
+          <stddev>0.01</stddev>
+        </noise>
+      </ray>
+      <gz_frame_id>lidar_r_link</gz_frame_id>
+      <topic>scan_right</topic>
+    </sensor>
+  </gazebo>
   </xacro:macro>
 </robot>

File: ffw_description/urdf/common/follower/ffw_follower_body.xacro (robot description, xacro)
@@ -63,8 +63,8 @@
          <inertial>
             <origin xyz="2.533965600e-02 0.000000000e+00 4.774514600e-02" />
-            <mass value="1.235180200e-01" />
-            <inertia ixx="6.870965700e-03" ixy="8.592260200e-07" ixz="-3.002664500e-04"
-            iyy="1.771510200e-02" iyz="-4.447973700e-07"
-            izz="1.631113500e-02" />
+            <mass value="0.123518" />
+            <inertia ixx="6.870965700e-06" ixy="8.592260200e-10" ixz="-3.002664500e-07"
+                     iyy="1.771510200e-05" iyz="-4.447973700e-10"
+                     izz="1.631113500e-05" />
          </inertial>
       </link>

File: ffw_description/urdf/ffw_sg2_rev1_follower/ffw_sg2_follower.urdf (robot description, URDF)
Before this commit: robot ffw_sg2_follower, 40 links, 39 joints
Links:
- link base_link: mass 3.598943900e+01 -> 35.989
- link lift_link: mass 1.790000000e+01 -> 17.9

File: ffw_description/urdf/ffw_sg2_rev1_follower/ffw_sg2_follower.urdf.xacro (robot description, xacro)
@@ -31,9 +31,10 @@
     </collision>
     <inertial>
-       <origin xyz="-4.574796400e-02 6.581058800e-03 1.943184200e-01" />
+       <!-- Center the base inertia to reduce biased yaw under straight motion -->
+       <origin xyz="0 0 0" />
        <mass value="3.598943900e+01" />
-       <inertia ixx="1.725473500e+04" ixy="6.471795500e-02" ixz="1.890204600e-01"
-       iyy="3.983747500e+04" iyz="1.716567300e-01"
-       izz="2.846139500e+04" />
+       <inertia ixx="1.725473500" ixy="6.471795500e-06" ixz="1.890204600e-05"
+       iyy="3.983747500" iyz="1.716567300e-05"
+       izz="2.846139500" />
     </inertial>
   </link>
@@ -44,4 +45,13 @@
   </joint>
   <link name="$(arg prefix)lidar_l_link">
+    <inertial>
+      <mass value="0.1"/>
+      <inertia ixx="0.0001" ixy="0" ixz="0" iyy="0.0001" iyz="0" izz="0.0001"/>
+    </inertial>
+    <visual>
+      <geometry>
+        <cylinder radius="0.03" length="0.03"/>
+      </geometry>
+    </visual>
   </link>
   <joint name="$(arg prefix)lidar_r_joint" type="fixed">
@@ -50,6 +60,6 @@
     <origin xyz="-0.111881 -0.240 0.34432" rpy="0 0 -1.57079632679"/>
   </joint>
-  <link name="$(arg prefix)lidar_r_link">
-  </link>
+  <!-- <link name="$(arg prefix)lidar_r_link">
+  </link> -->
   <joint name="$(arg prefix)imu_joint" type="fixed">
     <parent link="$(arg prefix)base_link"/>
@@ -59,4 +69,17 @@
   <link name="$(arg prefix)imu_link">
   </link>
+  <link name="$(arg prefix)lidar_r_link">
+    <inertial>
+      <mass value="0.1"/>
+      <origin xyz="0 0 0" rpy="0 0 0"/>
+      <inertia ixx="0.0001" ixy="0" ixz="0" iyy="0.0001" iyz="0" izz="0.0001"/>
+    </inertial>
+    <visual>
+      <geometry>
+        <cylinder radius="0.03" length="0.03"/>
+      </geometry>
+      <material name="blue"><color rgba="0 0 1 1"/></material>
+    </visual>
+  </link>
   <link name="$(arg prefix)lift_link">
     <visual>
@@ -77,8 +100,8 @@
     <inertial>
        <origin xyz="-1.286987800e-01 -1.604580800e-05 8.945601700e-01" />
-       <mass value="1.790000000e+01" />
-       <inertia ixx="1.009479700e+04" ixy="-3.568141800e-02" ixz="1.213165300e+03"
-       iyy="1.027057300e+04" iyz="7.021994000e-02"
-       izz="1.971602000e+02" />
+       <mass value="17.9" />
+       <inertia ixx="0.0100947" ixy="-0.0000000356" ixz="0.0012131"
+                iyy="0.0102705" iyz="0.0000000702"
+                izz="0.0001971" />
     </inertial>
   </link>
@@ -88,4 +111,6 @@
     <origin xyz="0.0 0.0 0.0" rpy="0 0 0"/>
   </joint>
+  <!-- Gazebo plugins/sensors -->
+  <xacro:ffw_sg2_follower_gazebo prefix="$(arg prefix)" />
   <xacro:ffw_follower_body parent="$(arg prefix)base_link" prefix="$(arg prefix)">
     <origin xyz="-0.0199 0 1.4316" rpy="0 0 0" />
@@ -177,8 +202,14 @@
       </material>
     </visual>
-    <collision>
+    <!-- <collision>
       <origin xyz="0 0 0" rpy="0 0 0" />
       <geometry>
         <mesh filename="${meshes_file_direction}/left_wheel_drive_link.stl" scale="0.001 0.001 0.001" />
+      </geometry>
+    </collision> -->
+    <collision>
+      <origin xyz="0 0 0" rpy="1.5708 0 0"/>
+      <geometry>
+        <cylinder radius="0.0865" length="0.05"/>
       </geometry>
     </collision>
@@ -239,8 +270,14 @@
       </material>
     </visual>
-    <collision>
+    <!-- <collision>
       <origin xyz="0 0 0" rpy="0 0 0" />
       <geometry>
         <mesh filename="${meshes_file_direction}/right_wheel_drive_link.stl" scale="0.001 0.001 0.001" />
+      </geometry>
+    </collision> -->
+    <collision>
+      <origin xyz="0 0 0" rpy="1.5708 0 0"/>
+      <geometry>
+        <cylinder radius="0.0865" length="0.05"/>
       </geometry>
     </collision>
@@ -302,9 +339,15 @@
     </visual>
     <collision>
+      <origin xyz="0 0 0" rpy="1.5708 0 0"/>
+      <geometry>
+        <cylinder radius="0.0865" length="0.05"/>
+      </geometry>
+    </collision>
+    <!-- <collision>
       <origin xyz="0 0 0" rpy="0 0 0" />
       <geometry>
         <mesh filename="${meshes_file_direction}/rear_wheel_drive_link.stl" scale="0.001 0.001 0.001" />
       </geometry>
-    </collision>
+    </collision> -->
     <inertial>
        <origin xyz="0.000000000e+00 1.499601700e-03 0.000000000e+00" />
