Commit message: Modified lift joint
Signed-off-by: Wonho Yun <ywh@robotis.com>

File: ffw_description/urdf/common/follower/ffw_follower_body.xacro (robot description, xacro)
@@ -13,5 +13,5 @@
          <dynamics damping="0.1" />
       </joint>
-      <joint name="${prefix}lift_joint" type="fixed">
+      <!-- <joint name="${prefix}lift_joint" type="fixed">
          <parent link="${parent}"/>
          <child link="${prefix}arm_base_link" />
@@ -20,5 +20,5 @@
          <limit velocity="4.8" effort="1000" lower="-0.5" upper="0.0" />
          <dynamics damping="0.1" />
-      </joint>
+      </joint> -->
       <link name="${prefix}arm_base_link">
          <visual>

Commit message: feat: Update hardware controller configurations for improved joint state handling and trajectory command broadcasting
Signed-off-by: Dongyun Kim <kdy@robotis.com>

File: ffw_description/urdf/common/follower/ffw_follower_body.xacro (robot description, xacro)
@@ -102,6 +102,6 @@
       </link>
       <xacro:zed_camera name="zedm" model="zedm" />
-      <joint name="zedm_joint" type="fixed">
-         <parent link="head_link2"/>
+      <joint name="${prefix}zedm_joint" type="fixed">
+         <parent link="${prefix}head_link2"/>
          <child link="zedm_camera_link"/>
          <origin xyz="0.0238122 -0.00651797 -0.0242094" rpy="0 0 0" />

File: ffw_description/urdf/ffw_bg2_rev4_follower/ffw_bg2_follower.urdf (robot description, URDF)
Before this commit: robot ffw_bg2_follower, 33 links, 32 joints
Links:
- added link zedm_camera_center; collision mesh filename=package://ffw_description/meshes/common/follower/zedm.stl scale=0.001 0.001 0.001; visual mesh filename=package://ffw_description/meshes/common/follower/zedm.stl scale=0.001 0.001 0.001
- added link zedm_camera_link
- added link zedm_left_camera_frame
- added link zedm_left_camera_optical_frame
- added link zedm_right_camera_frame
- added link zedm_right_camera_optical_frame
Joints:
- added joint zedm_camera_center_joint: type fixed, parent zedm_camera_link, child zedm_camera_center, origin xyz=0 0 0.01325 rpy=0 0 0
- added joint zedm_joint: type fixed, parent head_link2, child zedm_camera_link, origin xyz=0.0238122 -0.00651797 -0.0242094 rpy=0 0 0
- added joint zedm_left_camera_joint: type fixed, parent zedm_camera_center, child zedm_left_camera_frame, origin xyz=0 0.0315 0 rpy=0 0 0
- added joint zedm_left_camera_optical_joint: type fixed, parent zedm_left_camera_frame, child zedm_left_camera_optical_frame, origin xyz=0 0 0 rpy=-1.57079632679 0.0 -1.57079632679
- added joint zedm_right_camera_joint: type fixed, parent zedm_camera_center, child zedm_right_camera_frame, origin xyz=0 -0.0315 0 rpy=0 0 0
- added joint zedm_right_camera_optical_joint: type fixed, parent zedm_right_camera_frame, child zedm_right_camera_optical_frame, origin xyz=0 0 0 rpy=-1.57079632679 0.0 -1.57079632679

File: ffw_description/urdf/ffw_sg2_rev1_follower/ffw_sg2_follower.urdf (robot description, URDF)
Before this commit: robot ffw_sg2_follower, 40 links, 39 joints
Links:
- removed link world
- added link end_effector_l_link; visual box size=0.01 0.01 0.01
- added link end_effector_r_link; visual box size=0.01 0.01 0.01
- added link imu_link
- added link lidar_l_link
- added link lidar_r_link
- added link zedm_camera_center; collision mesh filename=file:///root/ros2_ws/install/ffw_description/share/ffw_desc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 scale=0.001 0.001 0.001; visual mesh filename=file:///root/ros2_ws/install/ffw_description/share/ffw_desc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 scale=0.001 0.001 0.001
- added link zedm_camera_link
- added link zedm_left_camera_frame
- added link zedm_left_camera_optical_frame
- added link zedm_right_camera_frame
- added link zedm_right_camera_optical_frame
Joints:
- removed joint world_fixed
- added joint end_effector_l_joint: type fixed, parent arm_l_link7, child end_effector_l_link, origin xyz=0 0 -0.215 rpy=0 0 0
- added joint end_effector_r_joint: type fixed, parent arm_r_link7, child end_effector_r_link, origin xyz=0 0 -0.215 rpy=0 0 0
- added joint imu_joint: type fixed, parent base_link, child imu_link, origin xyz=-0.1464 0.0 0.26 rpy=0 0 0
- added joint lidar_l_joint: type fixed, parent base_link, child lidar_l_link, origin xyz=-0.111881 0.240 0.34432 rpy=0 0 1.57079632679
- added joint lidar_r_joint: type fixed, parent base_link, child lidar_r_link, origin xyz=-0.111881 -0.240 0.34432 rpy=0 0 -1.57079632679
- added joint zedm_camera_center_joint: type fixed, parent zedm_camera_link, child zedm_camera_center, origin xyz=0 0 0.01325 rpy=0 0 0
- added joint zedm_joint: type fixed, parent head_link2, child zedm_camera_link, origin xyz=0.0238122 -0.00651797 -0.0242094 rpy=0 0 0
- added joint zedm_left_camera_joint: type fixed, parent zedm_camera_center, child zedm_left_camera_frame, origin xyz=0 0.0315 0 rpy=0 0 0
- added joint zedm_left_camera_optical_joint: type fixed, parent zedm_left_camera_frame, child zedm_left_camera_optical_frame, origin xyz=0 0 0 rpy=-1.57079632679 0.0 -1.57079632679
- added joint zedm_right_camera_joint: type fixed, parent zedm_camera_center, child zedm_right_camera_frame, origin xyz=0 -0.0315 0 rpy=0 0 0
- added joint zedm_right_camera_optical_joint: type fixed, parent zedm_right_camera_frame, child zedm_right_camera_optical_frame, origin xyz=0 0 0 rpy=-1.57079632679 0.0 -1.57079632679
- joint head_joint1: origin xyz=0.0494878 0 0.102123 rpy=0 0 0 -> xyz=0.049483 0 0.102130 rpy=0 0 0
- joint head_joint2: origin xyz=0.0365694 0 0.0563797 rpy=0 0 0 -> xyz=0.040 0 0.054 rpy=0 0 0
- joint left_wheel_drive: limit lower=-18.84955592153876 upper=18.84955592153876 effort=1 velocity=4.8 -> effort=9999.0 velocity=9999.0; type revolute -> continuous
- joint left_wheel_steer: limit lower=-18.84955592153876 upper=18.84955592153876 effort=1 velocity=4.8 -> lower=-18.84955592153876 upper=18.84955592153876 effort=9999.0 velocity=9999.0
- joint rear_wheel_drive: limit lower=-18.84955592153876 upper=18.84955592153876 effort=1 velocity=4.8 -> effort=9999.0 velocity=9999.0; type revolute -> continuous
- joint rear_wheel_steer: limit lower=-18.84955592153876 upper=18.84955592153876 effort=1 velocity=4.8 -> lower=-18.84955592153876 upper=18.84955592153876 effort=9999.0 velocity=9999.0
- joint right_wheel_drive: limit lower=-18.84955592153876 upper=18.84955592153876 effort=1 velocity=4.8 -> effort=9999.0 velocity=9999.0; type revolute -> continuous
- joint right_wheel_steer: limit lower=-18.84955592153876 upper=18.84955592153876 effort=1 velocity=4.8 -> lower=-18.84955592153876 upper=18.84955592153876 effort=9999.0 velocity=9999.0

Commit message: collsion test

File: ffw_description/urdf/common/follower/ffw_follower_body.xacro (robot description, xacro)
@@ -26,5 +26,5 @@
             <origin xyz="0 0 0" rpy="0 0 0" />
             <geometry>
-               <mesh filename="${meshes_file_direction}/body_arm_assy.stl" scale="0.001 0.001 0.001" />
+               <cylinder radius="0.08" length="0.15" />
             </geometry>
          </collision>
@@ -58,5 +58,5 @@
             <origin xyz="0 0 0" rpy="0 0 0" />
             <geometry>
-               <mesh filename="${meshes_file_direction}/head_link1.stl" scale="0.001 0.001 0.001" />
+               <cylinder radius="0.06" length="0.10" />
             </geometry>
          </collision>
@@ -90,5 +90,5 @@
             <origin xyz="0 0 0" rpy="0 0 0" />
             <geometry>
-               <mesh filename="${meshes_file_direction}/head_link2.stl" scale="0.001 0.001 0.001" />
+               <cylinder radius="0.05" length="0.08" />
             </geometry>
          </collision>
@@ -126,7 +126,7 @@
          </visual>
          <collision>
-            <origin xyz="0 0 0" rpy="0 0 0" />
-            <geometry>
-               <mesh filename="${meshes_file_direction}/arm_l_link1.stl" scale="0.001 0.001 0.001" />
+            <origin xyz="0 0.0615 0" rpy="0 0 0" />
+            <geometry>
+               <cylinder radius="0.04" length="0.123" />
             </geometry>
          </collision>
@@ -158,7 +158,7 @@
          </visual>
          <collision>
-            <origin xyz="0 0 0" rpy="0 0 0" />
-            <geometry>
-               <mesh filename="${meshes_file_direction}/arm_l_link2.stl" scale="0.001 0.001 0.001" />
+            <origin xyz="0 0 -0.0825" rpy="1.5708 0 0" />
+            <geometry>
+               <cylinder radius="0.04" length="0.165" />
             </geometry>
          </collision>
@@ -190,7 +190,7 @@
          </visual>
          <collision>
-            <origin xyz="0 0 0" rpy="0 0 0" />
-            <geometry>
-               <mesh filename="${meshes_file_direction}/arm_l_link3.stl" scale="0.001 0.001 0.001" />
+            <origin xyz="0.0205 0 -0.0825" rpy="0 0 0" />
+            <geometry>
+               <cylinder radius="0.035" length="0.135" />
             </geometry>
          </collision>
@@ -222,7 +222,7 @@
          </visual>
          <collision>
-            <origin xyz="0 0 0" rpy="0 0 0" />
-            <geometry>
-               <mesh filename="${meshes_file_direction}/arm_l_link4.stl" scale="0.001 0.001 0.001" />
+            <origin xyz="0 -0.0205 -0.07445" rpy="1.5708 0 0" />
+            <geometry>
+               <cylinder radius="0.035" length="0.1489" />
             </geometry>
          </collision>
@@ -254,7 +254,7 @@
          </visual>
          <collision>
-            <origin xyz="0 0 0" rpy="0 0 0" />
-            <geometry>
-               <mesh filename="${meshes_file_direction}/arm_l_link5.stl" scale="0.001 0.001 0.001" />
+            <origin xyz="0 0 -0.05205" rpy="0 0 0" />
+            <geometry>
+               <cylinder radius="0.03" length="0.1041" />
             </geometry>
          </collision>
@@ -286,7 +286,7 @@
          </visual>
          <collision>
-            <origin xyz="0 0 0" rpy="0 0 0" />
-            <geometry>
-               <mesh filename="${meshes_file_direction}/arm_l_link6.stl" scale="0.001 0.001 0.001" />
+            <origin xyz="0 0 -0.04425" rpy="1.5708 0 0" />
+            <geometry>
+               <cylinder radius="0.03" length="0.0885" />
             </geometry>
          </collision>
@@ -318,7 +318,7 @@
          </visual>
          <collision>
-            <origin xyz="0 0 0" rpy="0 0 0" />
-            <geometry>
-               <mesh filename="${meshes_file_direction}/arm_l_link7.stl" scale="0.001 0.001 0.001" />
+            <origin xyz="0.01275 0 -0.0277" rpy="0 0 0" />
+            <geometry>
+               <cylinder radius="0.025" length="0.055" />
             </geometry>
          </collision>
@@ -353,7 +353,7 @@
          </visual>
          <collision>
-            <origin xyz="0 0 0" rpy="0 0 0" />
-            <geometry>
-               <mesh filename="${meshes_file_direction}/arm_r_link1.stl" scale="0.001 0.001 0.001" />
+            <origin xyz="0 -0.0615 0" rpy="0 0 0" />
+            <geometry>
+               <cylinder radius="0.04" length="0.123" />
             </geometry>
          </collision>
@@ -385,7 +385,7 @@
          </visual>
          <collision>
-            <origin xyz="0 0 0" rpy="0 0 0" />
-            <geometry>
-               <mesh filename="${meshes_file_direction}/arm_r_link2.stl" scale="0.001 0.001 0.001" />
+            <origin xyz="0 0 -0.0825" rpy="1.5708 0 0" />
+            <geometry>
+               <cylinder radius="0.04" length="0.165" />
             </geometry>
          </collision>
@@ -417,7 +417,7 @@
          </visual>
          <collision>
-            <origin xyz="0 0 0" rpy="0 0 0" />
-            <geometry>
-               <mesh filename="${meshes_file_direction}/arm_r_link3.stl" scale="0.001 0.001 0.001" />
+            <origin xyz="0.0205 0 -0.0825" rpy="0 0 0" />
+            <geometry>
+               <cylinder radius="0.035" length="0.135" />
             </geometry>
          </collision>
@@ -449,7 +449,7 @@
          </visual>
          <collision>
-            <origin xyz="0 0 0" rpy="0 0 0" />
-            <geometry>
-               <mesh filename="${meshes_file_direction}/arm_r_link4.stl" scale="0.001 0.001 0.001" />
+            <origin xyz="0 -0.0205 -0.07445" rpy="1.5708 0 0" />
+            <geometry>
+               <cylinder radius="0.035" length="0.1489" />
             </geometry>
          </collision>
@@ -481,7 +481,7 @@
          </visual>
          <collision>
-            <origin xyz="0 0 0" rpy="0 0 0" />
-            <geometry>
-               <mesh filename="${meshes_file_direction}/arm_r_link5.stl" scale="0.001 0.001 0.001" />
+            <origin xyz="0 0 -0.05205" rpy="0 0 0" />
+            <geometry>
+               <cylinder radius="0.03" length="0.1041" />
             </geometry>
          </collision>
@@ -513,7 +513,7 @@
          </visual>
          <collision>
-            <origin xyz="0 0 0" rpy="0 0 0" />
-            <geometry>
-               <mesh filename="${meshes_file_direction}/arm_r_link6.stl" scale="0.001 0.001 0.001" />
+            <origin xyz="0 0 -0.04425" rpy="1.5708 0 0" />
+            <geometry>
+               <cylinder radius="0.03" length="0.0885" />
             </geometry>
          </collision>
@@ -545,7 +545,7 @@
          </visual>
          <collision>
-            <origin xyz="0 0 0" rpy="0 0 0" />
-            <geometry>
-               <mesh filename="${meshes_file_direction}/arm_r_link7.stl" scale="0.001 0.001 0.001" />
+            <origin xyz="0.01275 0 -0.0277" rpy="0 0 0" />
+            <geometry>
+               <cylinder radius="0.025" length="0.055" />
             </geometry>
          </collision>

File: ffw_description/urdf/common/follower/zedm.urdf.xacro (robot description, xacro)
@@ -14,7 +14,7 @@
 			</visual>
 			<collision>
-				<origin xyz="0 0 0" rpy="0 0 0"/>
+				<origin xyz="0 0 0.01325" rpy="0 0 0"/>
 				<geometry>
-					<mesh filename="file://$(find ffw_description)/meshes/common/follower/zedm.stl" scale="0.001 0.001 0.001"/>
+					<cylinder radius="0.04" length="0.12" />
 				</geometry>
 			</collision>

File: ffw_description/urdf/common/rh_p12_rn_a/rh_p12_rn_a.urdf.xacro (robot description, xacro)
@@ -14,7 +14,7 @@
     <link name="${prefix}rh_p12_rn_base">
       <collision>
-        <origin xyz="0 0 0" rpy="0 0 0"/>
+        <origin xyz="0 0 0.032" rpy="0 0 0"/>
         <geometry>
-          <mesh filename="${meshes_file_direction}/base.stl" scale="0.001 0.001 0.001"/>
+          <cylinder radius="0.03" length="0.064"/>
         </geometry>
       </collision>
@@ -46,7 +46,7 @@
     <link name="${prefix}rh_p12_rn_r1">
       <collision>
-        <origin xyz="0 0 0" rpy="0 0 0"/>
+        <origin xyz="0 0.034 0.004" rpy="0 0 0"/>
         <geometry>
-          <mesh filename="${meshes_file_direction}/r1.stl" scale="0.001 0.001 0.001"/>
+          <cylinder radius="0.015" length="0.068"/>
         </geometry>
       </collision>
@@ -79,7 +79,7 @@
     <link name="${prefix}rh_p12_rn_r2">
       <collision>
-        <origin xyz="0 0 0" rpy="0 0 0"/>
+        <origin xyz="0 0.006 0.011" rpy="0 0 0"/>
         <geometry>
-          <mesh filename="${meshes_file_direction}/r2.stl" scale="0.001 0.001 0.001"/>
+          <cylinder radius="0.01" length="0.022"/>
         </geometry>
       </collision>
@@ -112,7 +112,7 @@
     <link name="${prefix}rh_p12_rn_l1">
       <collision>
-        <origin xyz="0 0 0" rpy="0 0 0"/>
+        <origin xyz="0 -0.034 0.004" rpy="0 0 0"/>
         <geometry>
-          <mesh filename="${meshes_file_direction}/l1.stl" scale="0.001 0.001 0.001"/>
+          <cylinder radius="0.015" length="0.068"/>
         </geometry>
       </collision>
@@ -145,7 +145,7 @@
     <link name="${prefix}rh_p12_rn_l2">
       <collision>
-        <origin xyz="0 0 0" rpy="0 0 0"/>
+        <origin xyz="0 -0.006 0.011" rpy="0 0 0"/>
         <geometry>
-          <mesh filename="${meshes_file_direction}/l2.stl" scale="0.001 0.001 0.001"/>
+          <cylinder radius="0.01" length="0.022"/>
         </geometry>
       </collision>

File: ffw_description/urdf/ffw_sg2_rev1_follower/ffw_sg2_follower.urdf.xacro (robot description, xacro)
@@ -25,7 +25,7 @@
     </visual>
     <collision>
-      <origin xyz="0 0 0" rpy="0 0 0" />
-      <geometry>
-        <mesh filename="${meshes_file_direction}/base_mobile_assy.stl" scale="0.001 0.001 0.001" />
+      <origin xyz="0 0 0.194" rpy="0 0 0" />
+      <geometry>
+        <cylinder radius="0.25" length="0.39" />
       </geometry>
     </collision>
@@ -70,7 +70,7 @@
     </visual>
     <collision>
-      <origin xyz="0 0 0" rpy="0 0 0" />
-      <geometry>
-        <mesh filename="${meshes_file_direction}/lift_link.stl" scale="0.001 0.001 0.001" />
+      <origin xyz="0 0 0.895" rpy="0 0 0" />
+      <geometry>
+        <cylinder radius="0.15" length="1.79" />
       </geometry>
     </collision>
@@ -147,7 +147,7 @@
     </visual>
     <collision>
-      <origin xyz="0 0 0" rpy="0 0 0" />
-      <geometry>
-        <mesh filename="${meshes_file_direction}/left_wheel_steer_link.stl" scale="0.001 0.001 0.001" />
+      <origin xyz="0.0098 -0.0547 -0.1377" rpy="0 0 0" />
+      <geometry>
+        <cylinder radius="0.08" length="0.15" />
       </geometry>
     </collision>
@@ -178,7 +178,7 @@
     </visual>
     <collision>
-      <origin xyz="0 0 0" rpy="0 0 0" />
-      <geometry>
-        <mesh filename="${meshes_file_direction}/left_wheel_drive_link.stl" scale="0.001 0.001 0.001" />
+      <origin xyz="0 -0.0015 0" rpy="1.5708 0 0" />
+      <geometry>
+        <cylinder radius="0.15" length="0.08" />
       </geometry>
     </collision>
@@ -209,7 +209,7 @@
     </visual>
     <collision>
-      <origin xyz="0 0 0" rpy="0 0 0" />
-      <geometry>
-        <mesh filename="${meshes_file_direction}/right_wheel_steer_link.stl" scale="0.001 0.001 0.001" />
+      <origin xyz="0.0098 0.0547 -0.1377" rpy="0 0 0" />
+      <geometry>
+        <cylinder radius="0.08" length="0.15" />
       </geometry>
     </collision>
@@ -240,7 +240,7 @@
     </visual>
     <collision>
-      <origin xyz="0 0 0" rpy="0 0 0" />
-      <geometry>
-        <mesh filename="${meshes_file_direction}/right_wheel_drive_link.stl" scale="0.001 0.001 0.001" />
+      <origin xyz="0 0.0015 0" rpy="1.5708 0 0" />
+      <geometry>
+        <cylinder radius="0.15" length="0.08" />
       </geometry>
     </collision>
@@ -271,7 +271,7 @@
     </visual>
     <collision>
-      <origin xyz="0 0 0" rpy="0 0 0" />
-      <geometry>
-        <mesh filename="${meshes_file_direction}/rear_wheel_steer_link.stl" scale="0.001 0.001 0.001" />
+      <origin xyz="0.0098 0.0547 -0.1377" rpy="0 0 0" />
+      <geometry>
+        <cylinder radius="0.08" length="0.15" />
       </geometry>
     </collision>
@@ -302,7 +302,7 @@
     </visual>
     <collision>
-      <origin xyz="0 0 0" rpy="0 0 0" />
-      <geometry>
-        <mesh filename="${meshes_file_direction}/rear_wheel_drive_link.stl" scale="0.001 0.001 0.001" />
+      <origin xyz="0 0.0015 0" rpy="1.5708 0 0" />
+      <geometry>
+        <cylinder radius="0.15" length="0.08" />
       </geometry>
     </collision>
