Commit message: Added vr script for hand retargeting
Signed-off-by: Hyunwoo Nam <nhw@robotis.com>

File: ffw_description/urdf/common/hx5_d20/hx5_d20_right.urdf (robot description, URDF)
Before this commit: robot hx5_d20_right, 26 links, 25 joints
Joints:
- joint finger_r_joint_a: child ${prefix}finger_r_link1 -> finger_r_link1; parent ${prefix}hx5_d20_right_base -> hx5_d20_right_base
