Commit message: Fixed vr indent
Signed-off-by: Hyunwoo Nam <nhw@robotis.com>

File: ffw_description/urdf/common/hx5_d20/hx5_d20_left.urdf (robot description, URDF)
Before this commit: robot hx5_d20_left, 26 links, 25 joints
Joints:
- joint finger_l_joint_b: limit lower=0.0 upper=3.14 effort=1000 velocity=4.8 -> lower=0.0 upper=1.57 effort=1000 velocity=4.8

File: ffw_description/urdf/common/hx5_d20/hx5_d20_right.urdf (robot description, URDF)
Before this commit: robot hx5_d20_right, 26 links, 25 joints
Joints:
- joint finger_r_joint_b: limit lower=-3.14 upper=0.0 effort=1000 velocity=4.8 -> lower=-1.57 upper=0.0 effort=1000 velocity=4.8
