Commit message: Added end effector link to the palm of HX5-D20
Signed-off-by: Hyunwoo Nam <nhw@robotis.com>

File: ffw_description/urdf/common/hx5_d20/hx5_d20_left.urdf.xacro (robot description, xacro)
@@ -35,4 +35,20 @@
          </inertial>
       </link>
+      <joint name="${prefix}palm" type="fixed">
+         <parent link="${prefix}hx5_d20_left_base" />
+         <child link="end_effector_l_link" />
+         <origin xyz="0.0 0.0 0.054" rpy="0 0 0" />
+      </joint>
+      <link name="end_effector_l_link">
+         <visual>
+            <origin xyz="0 0 0" rpy="0 0 0"/>
+            <geometry>
+            <box size="0.01 0.01 0.01" />
+            </geometry>
+            <material name="red">
+            <color rgba="1.0 0.0 0.0 1"/>
+            </material>
+         </visual>
+      </link>
       <!-- THUMB -->
       <joint name="${prefix}finger_l_joint1" type="revolute">

File: ffw_description/urdf/common/hx5_d20/hx5_d20_right.urdf.xacro (robot description, xacro)
@@ -35,4 +35,20 @@
          </inertial>
       </link>
+      <joint name="${prefix}palm" type="fixed">
+         <parent link="${prefix}hx5_d20_right_base" />
+         <child link="end_effector_r_link" />
+         <origin xyz="0.0 0.0 0.054" rpy="0 0 0" />
+      </joint>
+      <link name="end_effector_r_link">
+         <visual>
+            <origin xyz="0 0 0" rpy="0 0 0"/>
+            <geometry>
+            <box size="0.01 0.01 0.01" />
+            </geometry>
+            <material name="red">
+            <color rgba="1.0 0.0 0.0 1"/>
+            </material>
+         </visual>
+      </link>
       <!-- THUMB -->
       <joint name="${prefix}finger_r_joint1" type="revolute">

Commit message: Fixed palm joint name
Signed-off-by: Hyunwoo Nam <nhw@robotis.com>

File: ffw_description/urdf/common/hx5_d20/hx5_d20_left.urdf.xacro (robot description, xacro)
@@ -35,5 +35,5 @@
          </inertial>
       </link>
-      <joint name="${prefix}palm" type="fixed">
+      <joint name="${prefix}l_palm" type="fixed">
          <parent link="${prefix}hx5_d20_left_base" />
          <child link="end_effector_l_link" />

File: ffw_description/urdf/common/hx5_d20/hx5_d20_right.urdf.xacro (robot description, xacro)
@@ -35,5 +35,5 @@
          </inertial>
       </link>
-      <joint name="${prefix}palm" type="fixed">
+      <joint name="${prefix}r_palm" type="fixed">
          <parent link="${prefix}hx5_d20_right_base" />
          <child link="end_effector_r_link" />
