Commit message: Refactor gravity compensation controller parameters and launch configurations to support optional spring effects. Update YAML and Xacro files to include new spring effect parameters, while commenting out legacy configurations for clarity. Adjust launch scripts to disable unused controllers.

File: ffw_description/ros2_control/ffw_lg2_rev3_leader/ffw_lg2_rev3_leader_current.ros2_control.xacro (robot description, xacro)
@@ -21,6 +21,6 @@
             <param name="baud_rate">4000000</param>
             <param name="dynamixel_model_folder">/param/dxl_model</param>
-            <param name="number_of_joints">16</param>
-            <param name="number_of_transmissions">16</param>
+            <param name="number_of_joints">8</param>
+            <param name="number_of_transmissions">8</param>
             <param name="disable_torque_at_init">true</param>
             <param name="dynamixel_state_pub_msg_name">dynamixel_hardware_interface/dxl_state</param>
@@ -32,5 +32,5 @@
         </hardware>
       </xacro:unless>
-      <sensor name="sensorxel_l_joy">
+      <!-- <sensor name="sensorxel_l_joy">
         <state_interface name="JOYSTICK X VALUE"/>
         <state_interface name="JOYSTICK Y VALUE"/>
@@ -83,5 +83,5 @@
         <state_interface name="velocity"/>
         <state_interface name="effort"/>
-      </joint>
+      </joint> -->
       <sensor name="sensorxel_r_joy">
         <state_interface name="JOYSTICK X VALUE"/>
@@ -136,5 +136,5 @@
         <state_interface name="effort"/>
       </joint>
-      <gpio name="sensorxel_l_joy">
+      <!-- <gpio name="sensorxel_l_joy">
         <param name="type">sensor</param>
         <param name="ID">40</param>
@@ -237,5 +237,5 @@
         <param name="Return Delay Time">0</param>
         <param name="Torque Enable">1</param>
-      </gpio>
+      </gpio> -->
       <gpio name="sensorxel_r_joy">
         <param name="type">sensor</param>
