Commit message: Removed end_effector TF between arm and hand
Signed-off-by: Hyunwoo Nam <nhw@robotis.com>

File: ffw_description/urdf/ffw_sh5_rev1_follower/ffw_sh5_follower.urdf (robot description, URDF)
Before this commit: robot ffw_sh5_follower, 92 links, 91 joints
Links:
- removed link end_effector_l_link
- removed link end_effector_r_link
Joints:
- removed joint end_effector_l_joint
- removed joint end_effector_r_joint

File: ffw_description/urdf/ffw_sh5_rev1_follower/ffw_sh5_follower.urdf.xacro (robot description, xacro)
@@ -97,36 +97,4 @@
     <origin xyz="0 0 -0.078" rpy="0 3.14159265359 -1.5708"/>
   </xacro:hx5_d20_right>
-  <joint name="$(arg prefix)end_effector_l_joint" type="fixed">
-    <parent link="$(arg prefix)arm_l_link7"/>
-    <child link="$(arg prefix)end_effector_l_link"/>
-    <origin xyz="0 0 -0.215" rpy="0 0 0"/>
-  </joint>
-  <link name="$(arg prefix)end_effector_l_link">
-    <visual>
-      <origin xyz="0 0 0" rpy="0 0 0"/>
-      <geometry>
-        <box size="0.01 0.01 0.01" />
-      </geometry>
-      <material name="red">
-        <color rgba="1.0 0.0 0.0 1"/>
-      </material>
-    </visual>
-  </link>
-  <joint name="$(arg prefix)end_effector_r_joint" type="fixed">
-    <parent link="$(arg prefix)arm_r_link7"/>
-    <child link="$(arg prefix)end_effector_r_link"/>
-    <origin xyz="0 0 -0.215" rpy="0 0 0"/>
-  </joint>
-  <link name="$(arg prefix)end_effector_r_link">
-    <visual>
-      <origin xyz="0 0 0" rpy="0 0 0"/>
-      <geometry>
-        <box size="0.01 0.01 0.01" />
-      </geometry>
-      <material name="red">
-        <color rgba="1.0 0.0 0.0 1"/>
-      </material>
-    </visual>
-  </link>
   <joint name="$(arg prefix)left_wheel_steer" type="revolute">
       <parent link="$(arg prefix)base_link"/>

Commit message: Fixed swerve drive inertial values
Signed-off-by: Hyunwoo Nam <nhw@robotis.com>

File: ffw_description/urdf/ffw_sh5_rev1_follower/ffw_sh5_follower.urdf (robot description, URDF)
Before this commit: robot ffw_sh5_follower, 90 links, 89 joints
Links:
- link base_link: mass 3.598943900e+01 -> 35.989

File: ffw_description/urdf/ffw_sh5_rev1_follower/ffw_sh5_follower.urdf.xacro (robot description, xacro)
@@ -31,9 +31,10 @@
     </collision>
     <inertial>
-       <origin xyz="-4.574796400e-02 6.581058800e-03 1.943184200e-01" />
+       <!-- Center the base inertia to reduce biased yaw under straight motion -->
+       <origin xyz="0 0 0" />
        <mass value="3.598943900e+01" />
-       <inertia ixx="1.725473500e+04" ixy="6.471795500e-02" ixz="1.890204600e-01"
-       iyy="3.983747500e+04" iyz="1.716567300e-01"
-       izz="2.846139500e+04" />
+       <inertia ixx="1.725473500" ixy="6.471795500e-06" ixz="1.890204600e-05"
+       iyy="3.983747500" iyz="1.716567300e-05"
+       izz="2.846139500" />
     </inertial>
   </link>
@@ -77,8 +78,8 @@
     <inertial>
        <origin xyz="-1.286987800e-01 -1.604580800e-05 8.945601700e-01" />
-       <mass value="1.790000000e+01" />
-       <inertia ixx="1.009479700e+04" ixy="-3.568141800e-02" ixz="1.213165300e+03"
-       iyy="1.027057300e+04" iyz="7.021994000e-02"
-       izz="1.971602000e+02" />
+       <mass value="17.9" />
+       <inertia ixx="0.0100947" ixy="-0.0000000356" ixz="0.0012131"
+                iyy="0.0102705" iyz="0.0000000702"
+                izz="0.0001971" />
     </inertial>
   </link>
@@ -145,8 +146,14 @@
       </material>
     </visual>
-    <collision>
+    <!-- <collision>
       <origin xyz="0 0 0" rpy="0 0 0" />
       <geometry>
         <mesh filename="${meshes_file_direction}/left_wheel_drive_link.stl" scale="0.001 0.001 0.001" />
+      </geometry>
+    </collision> -->
+    <collision>
+      <origin xyz="0 0 0" rpy="1.5708 0 0"/>
+      <geometry>
+        <cylinder radius="0.0865" length="0.05"/>
       </geometry>
     </collision>
@@ -207,8 +214,14 @@
       </material>
     </visual>
-    <collision>
+    <!-- <collision>
       <origin xyz="0 0 0" rpy="0 0 0" />
       <geometry>
         <mesh filename="${meshes_file_direction}/right_wheel_drive_link.stl" scale="0.001 0.001 0.001" />
+      </geometry>
+    </collision> -->
+    <collision>
+      <origin xyz="0 0 0" rpy="1.5708 0 0"/>
+      <geometry>
+        <cylinder radius="0.0865" length="0.05"/>
       </geometry>
     </collision>
@@ -269,8 +282,14 @@
       </material>
     </visual>
-    <collision>
+    <!-- <collision>
       <origin xyz="0 0 0" rpy="0 0 0" />
       <geometry>
         <mesh filename="${meshes_file_direction}/rear_wheel_drive_link.stl" scale="0.001 0.001 0.001" />
+      </geometry>
+    </collision> -->
+    <collision>
+      <origin xyz="0 0 0" rpy="1.5708 0 0"/>
+      <geometry>
+        <cylinder radius="0.0865" length="0.05"/>
       </geometry>
     </collision>
