Commit message: Removed commented block
Signed-off-by: Hyunwoo Nam <nhw@robotis.com>

File: ffw_description/urdf/ffw_sh5_rev1_follower/ffw_sh5_follower.urdf.xacro (robot description, xacro)
@@ -302,40 +302,4 @@
     </inertial>
   </link>
-  <!-- <joint name="$(arg prefix)gripper_r_joint1" type="revolute">
-    <parent link="$(arg prefix)base_link" />
-    <child link="$(arg prefix)dummy_link1" />
-    <origin xyz="0.0 0.0 0.0" rpy="0 0 0" />
-    <limit effort="1000" lower="-0.2317" upper="0.6951" velocity="4.8"/>
-    <dynamics damping="0.1"/>
-  </joint>
-  <link name="$(arg prefix)dummy_link1">
-      <visual>
-        <origin xyz="0 0 0" rpy="0 0 0"/>
-        <geometry>
-        <box size="0.01 0.01 0.01" />
-        </geometry>
-        <material name="red">
-        <color rgba="1.0 0.0 0.0 1"/>
-        </material>
-      </visual>
-  </link>
-  <joint name="$(arg prefix)gripper_l_joint1" type="revolute">
-    <parent link="$(arg prefix)base_link" />
-    <child link="$(arg prefix)dummy_link2" />
-    <origin xyz="0.0 0.0 0.0" rpy="0 0 0" />
-    <limit effort="1000" lower="-0.2317" upper="0.6951" velocity="4.8"/>
-    <dynamics damping="0.1"/>
-  </joint>
-  <link name="$(arg prefix)dummy_link2">
-      <visual>
-        <origin xyz="0 0 0" rpy="0 0 0"/>
-        <geometry>
-        <box size="0.01 0.01 0.01" />
-        </geometry>
-        <material name="red">
-        <color rgba="1.0 0.0 0.0 1"/>
-        </material>
-      </visual>
-  </link> -->
   <xacro:ffw_sh5_follower_system
     use_sim="$(arg use_sim)"
