Commit message: Modified link7 mesh and inertia

File: ffw_description/urdf/common/leader/ffw_mini_leader_body.urdf.xacro (robot description, xacro)
@@ -567,13 +567,13 @@
          </collision>
          <inertial>
-            <origin xyz="-0.047248892 0.0065185210 -0.086220290" rpy="0 0 0" />
+            <origin xyz="-0.047110855 0.0067030274 -0.086068978" rpy="0 0 0" />
             <mass value="0.30067384" />
             <inertia
-               ixx="0.00048973350"
-               ixy="-0.000038599418"
-               ixz="0.000048657081"
-               iyy="0.00093764064"
-               iyz="0.000061401720"
-               izz="0.00055518610" />
+               ixx="0.00048869771"
+               ixy="-0.000040597374"
+               ixz="0.000048513897"
+               iyy="0.00093640099"
+               iyz="0.000061136258"
+               izz="0.00055404990" />
          </inertial>
       </link>
