Commit message: Modified for sh5

File: ffw_description/ros2_control/ffw_sh5_rev1_follower/ffw_sh5_follower.ros2_control.xacro (robot description, xacro)
@@ -20,6 +20,6 @@
             <param name="baud_rate">4000000</param>
             <param name="dynamixel_model_folder">/param/dxl_model</param>
-            <param name="number_of_joints">57</param>
-            <param name="number_of_transmissions">57</param>
+            <param name="number_of_joints">60</param>
+            <param name="number_of_transmissions">60</param>
             <param name="disable_torque_at_init">true</param>
             <param name="dynamixel_state_pub_msg_name">dynamixel_hardware_interface/dxl_state</param>
@@ -505,4 +505,10 @@
         <state_interface name="effort"/>
       </joint>
+      <joint name="lift_joint">
+        <command_interface name="position"/>
+        <state_interface name="position"/>
+        <state_interface name="velocity"/>
+        <state_interface name="effort"/>
+      </joint>
       <joint name="head_joint1">
         <command_interface name="position"/>
@@ -517,5 +523,17 @@
         <state_interface name="effort"/>
       </joint>
-      <joint name="lift_joint">
+      <joint name="left_wheel_steer">
+        <command_interface name="position"/>
+        <state_interface name="position"/>
+        <state_interface name="velocity"/>
+        <state_interface name="effort"/>
+      </joint>
+      <joint name="right_wheel_steer">
+        <command_interface name="position"/>
+        <state_interface name="position"/>
+        <state_interface name="velocity"/>
+        <state_interface name="effort"/>
+      </joint>
+      <joint name="rear_wheel_steer">
         <command_interface name="position"/>
         <state_interface name="position"/>
@@ -2631,47 +2649,4 @@
         <param name="Min Position Limit">-151875</param>
       </gpio>
-      <!-- HEAD -->
-      <gpio name="dxl61">
-        <param name="type">dxl</param>
-        <param name="ID">61</param>z
-        <command_interface name="Goal Position"/>
-        <state_interface name="Present Position"/>
-        <state_interface name="Present Velocity"/>
-        <state_interface name="Present Current"/>
-        <state_interface name="Hardware Error Status"/>
-        <param name="Drive Mode">1</param>
-        <param name="Operating Mode">3</param>
-        <param name="Return Delay Time">0</param>
-        <param name="Profile Velocity">100</param>
-        <param name="Profile Acceleration">50</param>
-        <param name="Max Position Limit">2500</param>
-        <param name="Min Position Limit">1896</param>
-        <param name="Position P Gain">1600</param>
-        <param name="Position I Gain">400</param>
-        <param name="Position D Gain">400</param>
-        <param name="Feedforward 1st Gain">30</param>
-        <param name="Feedforward 2nd Gain">30</param>
-      </gpio>
-      <gpio name="dxl62">
-        <param name="type">dxl</param>
-        <param name="ID">62</param>
-        <command_interface name="Goal Position"/>
-        <state_interface name="Present Position"/>
-        <state_interface name="Present Velocity"/>
-        <state_interface name="Present Current"/>
-        <state_interface name="Hardware Error Status"/>
-        <param name="Drive Mode">1</param>
-        <param name="Operating Mode">3</param>
-        <param name="Return Delay Time">0</param>
-        <param name="Profile Velocity">100</param>
-        <param name="Profile Acceleration">50</param>
-        <param name="Max Position Limit">2275</param>
-        <param name="Min Position Limit">1820</param>
-        <param name="Position P Gain">800</param>
-        <param name="Position I Gain">200</param>
-        <param name="Position D Gain">200</param>
-        <param name="Feedforward 1st Gain">30</param>
-        <param name="Feedforward 2nd Gain">30</param>
-      </gpio>
       <!-- LIFT -->
       <gpio name="dxl81">
@@ -2697,4 +2672,110 @@
         <param name="Velocity P Gain">41387</param>
         <param name="Velocity I Gain">1065630</param>
+      </gpio>
+      <!-- HEAD -->
+      <gpio name="dxl61">
+        <param name="type">dxl</param>
+        <param name="ID">61</param>z
+        <command_interface name="Goal Position"/>
+        <state_interface name="Present Position"/>
+        <state_interface name="Present Velocity"/>
+        <state_interface name="Present Current"/>
+        <state_interface name="Hardware Error Status"/>
+        <param name="Drive Mode">1</param>
+        <param name="Operating Mode">3</param>
+        <param name="Return Delay Time">0</param>
+        <param name="Profile Velocity">100</param>
+        <param name="Profile Acceleration">50</param>
+        <param name="Max Position Limit">2500</param>
+        <param name="Min Position Limit">1896</param>
+        <param name="Position P Gain">1600</param>
+        <param name="Position I Gain">400</param>
+        <param name="Position D Gain">400</param>
+        <param name="Feedforward 1st Gain">30</param>
+        <param name="Feedforward 2nd Gain">30</param>
+      </gpio>
+      <gpio name="dxl62">
+        <param name="type">dxl</param>
+        <param name="ID">62</param>
+        <command_interface name="Goal Position"/>
+        <state_interface name="Present Position"/>
+        <state_interface name="Present Velocity"/>
+        <state_interface name="Present Current"/>
+        <state_interface name="Hardware Error Status"/>
+        <param name="Drive Mode">1</param>
+        <param name="Operating Mode">3</param>
+        <param name="Return Delay Time">0</param>
+        <param name="Profile Velocity">100</param>
+        <param name="Profile Acceleration">50</param>
+        <param name="Max Position Limit">2275</param>
+        <param name="Min Position Limit">1820</param>
+        <param name="Position P Gain">800</param>
+        <param name="Position I Gain">200</param>
+        <param name="Position D Gain">200</param>
+        <param name="Feedforward 1st Gain">30</param>
+        <param name="Feedforward 2nd Gain">30</param>
+      </gpio>
+      <!-- LEFT WHEEL -->
+      <gpio name="dxl101">
+        <param name="type">dxl</param>
+        <param name="ID">101</param>
+        <command_interface name="Goal Position"/>
+        <state_interface name="Present Position"/>
+        <state_interface name="Present Velocity"/>
+        <state_interface name="Present Current"/>
+        <state_interface name="Error Code"/>
+        <param name="Drive Mode">5</param>
+        <param name="Operating Mode">3</param>
+        <param name="Velocity Limit">12592</param>
+        <param name="Acceleration Limit">125920</param>
+        <param name="Min Position Limit">-1572864</param>
+        <param name="Max Position Limit">1572864</param>
+        <param name="Acceleration Limit">1010</param>
+        <param name="Return Delay Time">0</param>
+        <param name="Profile Velocity">12592</param>
+        <param name="Profile Acceleration Time">500</param>
+        <param name="Profile Time">1000</param>
+      </gpio>
+      <!-- RIGHT WHEEL -->
+      <gpio name="dxl103">
+        <param name="type">dxl</param>
+        <param name="ID">103</param>
+        <command_interface name="Goal Position"/>
+        <state_interface name="Present Position"/>
+        <state_interface name="Present Velocity"/>
+        <state_interface name="Present Current"/>
+        <state_interface name="Error Code"/>
+        <param name="Drive Mode">5</param>
+        <param name="Operating Mode">3</param>
+        <param name="Velocity Limit">12592</param>
+        <param name="Acceleration Limit">125920</param>
+        <param name="Min Position Limit">-1572864</param>
+        <param name="Max Position Limit">1572864</param>
+        <param name="Acceleration Limit">1010</param>
+        <param name="Return Delay Time">0</param>
+        <param name="Profile Velocity">12592</param>
+        <param name="Profile Acceleration Time">500</param>
+        <param name="Profile Time">1000</param>
+      </gpio>
+      <!-- REAR WHEEL -->
+      <gpio name="dxl105">
+        <param name="type">dxl</param>
+        <param name="ID">105</param>
+        <command_interface name="Goal Position"/>
+        <state_interface name="Present Position"/>
+        <state_interface name="Present Velocity"/>
+        <state_interface name="Present Current"/>
+        <state_interface name="Error Code"/>
+        <param name="Drive Mode">5</param>
+        <param name="Operating Mode">3</param>
+        <param name="Velocity Limit">12592</param>
+        <param name="Acceleration Limit">125920</param>
+        <param name="Min Position Limit">-1572864</param>
+        <param name="Max Position Limit">1572864</param>
+        <param name="Acceleration Limit">1010</param>
+        <param name="Return Delay Time">0</param>
+        <param name="Profile Velocity">12592</param>
+        <param name="Profile Acceleration Time">500</param>
+        <param name="Profile Time">1000</param>
       </gpio>
     </ros2_control>
