Commit message: Modified for sh5

File: ffw_description/urdf/ffw_sh5_rev1_follower/ffw_sh5_follower.urdf.xacro (robot description, xacro)
@@ -11,37 +11,83 @@
   <xacro:include filename="$(find ffw_description)/urdf/common/hx5_d20_right/hx5_d20_right.urdf.xacro" />
   <xacro:include filename="$(find ffw_description)/ros2_control/$(arg model)/ffw_sh5_follower.ros2_control.xacro" />
+  <xacro:include filename="$(find ffw_description)/ros2_control/$(arg model)/ffw_sh5_base.ros2_control.xacro" />
+  <xacro:include filename="$(find ffw_description)/ros2_control/$(arg model)/ffw_sh5_sensor.ros2_control.xacro" />
   <xacro:include filename="$(find ffw_description)/gazebo/ffw_sh5_rev1_follower/ffw_sh5_follower.gazebo.xacro" />
-  <link name="world"/>
-  <joint name="$(arg prefix)world_fixed" type="fixed">
-    <parent link="world"/>
-    <child link="$(arg prefix)base_link"/>
+  <link name="$(arg prefix)base_link">
+    <visual>
+      <origin xyz="0 0 0" rpy="0 0 0" />
+      <geometry>
+        <mesh filename="${meshes_file_direction}/base_mobile_assy.stl" scale="0.001 0.001 0.001" />
+      </geometry>
+      <material name="silver">
+        <color rgba="0.75 0.75 0.75 1"/>
+      </material>
+    </visual>
+    <collision>
+      <origin xyz="0 0 0" rpy="0 0 0" />
+      <geometry>
+        <mesh filename="${meshes_file_direction}/base_mobile_assy.stl" scale="0.001 0.001 0.001" />
+      </geometry>
+    </collision>
+    <inertial>
+       <origin xyz="-4.574796400e-02 6.581058800e-03 1.943184200e-01" />
+       <mass value="3.598943900e+01" />
+       <inertia ixx="1.725473500e+04" ixy="6.471795500e-02" ixz="1.890204600e-01"
+       iyy="3.983747500e+04" iyz="1.716567300e-01"
+       izz="2.846139500e+04" />
+    </inertial>
+  </link>
+  <joint name="$(arg prefix)lidar_l_joint" type="fixed">
+    <parent link="$(arg prefix)base_link"/>
+    <child link="$(arg prefix)lidar_l_link"/>
+    <origin xyz="-0.111881 0.240 0.34432" rpy="0 0 1.57079632679"/>
+  </joint>
+  <link name="$(arg prefix)lidar_l_link">
+  </link>
+  <joint name="$(arg prefix)lidar_r_joint" type="fixed">
+    <parent link="$(arg prefix)base_link"/>
+    <child link="$(arg prefix)lidar_r_link"/>
+    <origin xyz="-0.111881 -0.240 0.34432" rpy="0 0 -1.57079632679"/>
+  </joint>
+  <link name="$(arg prefix)lidar_r_link">
+  </link>
+  <joint name="$(arg prefix)imu_joint" type="fixed">
+    <parent link="$(arg prefix)base_link"/>
+    <child link="$(arg prefix)imu_link"/>
+    <origin xyz="-0.1464 0.0 0.26" rpy="0 0 0"/>
+  </joint>
+  <link name="$(arg prefix)imu_link">
+  </link>
+  <link name="$(arg prefix)lift_link">
+    <visual>
+      <origin xyz="0 0 0" rpy="0 0 0" />
+      <geometry>
+        <mesh filename="${meshes_file_direction}/lift_link.stl" scale="0.001 0.001 0.001" />
+      </geometry>
+      <material name="silver">
+        <color rgba="0.75 0.75 0.75 1"/>
+      </material>
+    </visual>
+    <collision>
+      <origin xyz="0 0 0" rpy="0 0 0" />
+      <geometry>
+        <mesh filename="${meshes_file_direction}/lift_link.stl" scale="0.001 0.001 0.001" />
+      </geometry>
+    </collision>
+    <inertial>
+       <origin xyz="-1.286987800e-01 -1.604580800e-05 8.945601700e-01" />
+       <mass value="1.790000000e+01" />
+       <inertia ixx="1.009479700e+04" ixy="-3.568141800e-02" ixz="1.213165300e+03"
+       iyy="1.027057300e+04" iyz="7.021994000e-02"
+       izz="1.971602000e+02" />
+    </inertial>
+  </link>
+  <joint name="$(arg prefix)lift_fixed_joint" type="fixed">
+    <parent link="$(arg prefix)base_link"/>
+    <child link="$(arg prefix)lift_link"/>
     <origin xyz="0.0 0.0 0.0" rpy="0 0 0"/>
   </joint>
-  <link name="$(arg prefix)base_link">
-    <visual>
-      <origin xyz="0 0 0" rpy="0 0 0" />
-      <geometry>
-        <mesh filename="${meshes_file_direction}/base_mobile_assy.stl" scale="0.001 0.001 0.001" />
-      </geometry>
-      <material name="silver">
-        <color rgba="0.75 0.75 0.75 1"/>
-      </material>
-    </visual>
-    <collision>
-      <origin xyz="0 0 0" rpy="0 0 0" />
-      <geometry>
-        <mesh filename="${meshes_file_direction}/base_mobile_assy.stl" scale="0.001 0.001 0.001" />
-      </geometry>
-    </collision>
-    <inertial>
-      <origin xyz="-8.880608700e-03 -4.758427800e-03 3.886366400e-01" />
-      <mass value="5.435831600e+01" />
-      <inertia ixx="1.188633900e+06" ixy="6.334393100e+02" ixz="-1.454811600e+05"
-      iyy="1.090949100e+06" iyz="-5.126785200e+03"
-      izz="4.492808000e+05" />
-    </inertial>
-  </link>
   <xacro:ffw_follower_body parent="$(arg prefix)base_link" prefix="$(arg prefix)">
-    <origin xyz="0.0055 0 1.4316" rpy="0 0 0" />
+    <origin xyz="-0.0199 0 1.4316" rpy="0 0 0" />
   </xacro:ffw_follower_body>
   <xacro:hx5_d20_left parent="$(arg prefix)arm_l_link7" prefix="$(arg prefix)">
@@ -51,8 +97,222 @@
     <origin xyz="0 0 -0.078" rpy="0 3.14159265359 -1.5708"/>
   </xacro:hx5_d20_right>
-  <xacro:ffw_sh5_follower_system
-    use_sim="$(arg use_sim)"
-    use_mock_hardware="$(arg use_mock_hardware)"
-    mock_sensor_commands="$(arg mock_sensor_commands)"/>
+  <joint name="$(arg prefix)end_effector_l_joint" type="fixed">
+    <parent link="$(arg prefix)arm_l_link7"/>
+    <child link="$(arg prefix)end_effector_l_link"/>
+    <origin xyz="0 0 -0.215" rpy="0 0 0"/>
+  </joint>
+  <link name="$(arg prefix)end_effector_l_link">
+    <visual>
+      <origin xyz="0 0 0" rpy="0 0 0"/>
+      <geometry>
+        <box size="0.01 0.01 0.01" />
+      </geometry>
+      <material name="red">
+        <color rgba="1.0 0.0 0.0 1"/>
+      </material>
+    </visual>
+  </link>
+  <joint name="$(arg prefix)end_effector_r_joint" type="fixed">
+    <parent link="$(arg prefix)arm_r_link7"/>
+    <child link="$(arg prefix)end_effector_r_link"/>
+    <origin xyz="0 0 -0.215" rpy="0 0 0"/>
+  </joint>
+  <link name="$(arg prefix)end_effector_r_link">
+    <visual>
+      <origin xyz="0 0 0" rpy="0 0 0"/>
+      <geometry>
+        <box size="0.01 0.01 0.01" />
+      </geometry>
+      <material name="red">
+        <color rgba="1.0 0.0 0.0 1"/>
+      </material>
+    </visual>
+  </link>
+  <joint name="$(arg prefix)left_wheel_steer" type="revolute">
+      <parent link="$(arg prefix)base_link"/>
+      <child link="$(arg prefix)left_wheel_steer_link"/>
+      <origin xyz="0.1371 0.2554 0.27555" rpy="0 0 0"/>
+      <axis xyz="0 0 1" />
+      <limit velocity="9999.0" effort="9999.0" lower="${-pi*6.0}" upper="${pi*6.0}" />
+  </joint>
+  <link name="$(arg prefix)left_wheel_steer_link">
+    <visual>
+      <origin xyz="0 0 0" rpy="0 0 0" />
+      <geometry>
+        <mesh filename="${meshes_file_direction}/left_wheel_steer_link.stl" scale="0.001 0.001 0.001" />
+      </geometry>
+      <material name="silver">
+        <color rgba="0.75 0.75 0.75 1"/>
+      </material>
+    </visual>
+    <collision>
+      <origin xyz="0 0 0" rpy="0 0 0" />
+      <geometry>
+        <mesh filename="${meshes_file_direction}/left_wheel_steer_link.stl" scale="0.001 0.001 0.001" />
+      </geometry>
+    </collision>
+    <inertial>
+       <origin xyz="9.802769300e-03 -5.471240900e-02 -1.376533800e-01" />
+       <mass value="7.550951000e-01" />
+       <inertia ixx="2.797326600e-03" ixy="-3.290807800e-05" ixz="-1.950671800e-04"
+       iyy="3.582264900e-03" iyz="-2.853290700e-04"
+       izz="1.683594000e-03" />
+    </inertial>
+  </link>
+  <joint name="$(arg prefix)left_wheel_drive" type="continuous">
+      <parent link="$(arg prefix)left_wheel_steer_link"/>
+      <child link="$(arg prefix)left_wheel_drive_link"/>
+      <origin xyz="0 0 -0.18905" rpy="0 0 0"/>
+      <axis xyz="0 1 0" />
+      <limit velocity="9999.0" effort="9999.0"/>
+  </joint>
+  <link name="$(arg prefix)left_wheel_drive_link">
+    <visual>
+      <origin xyz="0 0 0" rpy="0 0 0" />
+      <geometry>
+        <mesh filename="${meshes_file_direction}/left_wheel_drive_link.stl" scale="0.001 0.001 0.001" />
+      </geometry>
+      <material name="silver">
+        <color rgba="0.75 0.75 0.75 1"/>
+      </material>
+    </visual>
+    <collision>
+      <origin xyz="0 0 0" rpy="0 0 0" />
+      <geometry>
+        <mesh filename="${meshes_file_direction}/left_wheel_drive_link.stl" scale="0.001 0.001 0.001" />
+      </geometry>
+    </collision>
+    <inertial>
+       <origin xyz="0.000000000e+00 -1.499601700e-03 0.000000000e+00" />
+       <mass value="3.795460500e+00" />
+       <inertia ixx="7.187881500e-03" ixy="0.000000000e+00" ixz="0.000000000e+00"
+       iyy="1.156399900e-02" iyz="0.000000000e+00"
+       izz="7.187977000e-03" />
+    </inertial>
+  </link>
+  <joint name="$(arg prefix)right_wheel_steer" type="revolute">
+      <parent link="$(arg prefix)base_link"/>
+      <child link="$(arg prefix)right_wheel_steer_link"/>
+      <origin xyz="0.1371 -0.2554 0.27555" rpy="0 0 0"/>
+      <axis xyz="0 0 1" />
+      <limit velocity="9999.0" effort="9999.0" lower="${-pi*6.0}" upper="${pi*6.0}" />
+  </joint>
+  <link name="$(arg prefix)right_wheel_steer_link">
+    <visual>
+      <origin xyz="0 0 0" rpy="0 0 0" />
+      <geometry>
+        <mesh filename="${meshes_file_direction}/right_wheel_steer_link.stl" scale="0.001 0.001 0.001" />
+      </geometry>
+      <material name="silver">
+        <color rgba="0.75 0.75 0.75 1"/>
+      </material>
+    </visual>
+    <collision>
+      <origin xyz="0 0 0" rpy="0 0 0" />
+      <geometry>
+        <mesh filename="${meshes_file_direction}/right_wheel_steer_link.stl" scale="0.001 0.001 0.001" />
+      </geometry>
+    </collision>
+    <inertial>
+       <origin xyz="9.802728600e-03 5.471240900e-02 -1.376533400e-01" />
+       <mass value="7.550951000e-01" />
+       <inertia ixx="2.797322900e-03" ixy="3.290833300e-05" ixz="-1.950642500e-04"
+       iyy="3.582262300e-03" iyz="2.853288400e-04"
+       izz="1.683595100e-03" />
+    </inertial>
+  </link>
+  <joint name="$(arg prefix)right_wheel_drive" type="continuous">
+      <parent link="$(arg prefix)right_wheel_steer_link"/>
+      <child link="$(arg prefix)right_wheel_drive_link"/>
+      <origin xyz="0 0 -0.18905" rpy="0 0 0"/>
+      <axis xyz="0 1 0" />
+      <limit velocity="9999.0" effort="9999.0"/>
+  </joint>
+  <link name="$(arg prefix)right_wheel_drive_link">
+    <visual>
+      <origin xyz="0 0 0" rpy="0 0 0" />
+      <geometry>
+        <mesh filename="${meshes_file_direction}/right_wheel_drive_link.stl" scale="0.001 0.001 0.001" />
+      </geometry>
+      <material name="silver">
+        <color rgba="0.75 0.75 0.75 1"/>
+      </material>
+    </visual>
+    <collision>
+      <origin xyz="0 0 0" rpy="0 0 0" />
+      <geometry>
+        <mesh filename="${meshes_file_direction}/right_wheel_drive_link.stl" scale="0.001 0.001 0.001" />
+      </geometry>
+    </collision>
+    <inertial>
+       <origin xyz="0.000000000e+00 1.499601700e-03 0.000000000e+00" />
+       <mass value="3.795460500e+00" />
+       <inertia ixx="7.187881500e-03" ixy="0.000000000e+00" ixz="0.000000000e+00"
+       iyy="1.156399900e-02" iyz="0.000000000e+00"
+       izz="7.187977000e-03" />
+    </inertial>
+  </link>
+  <joint name="$(arg prefix)rear_wheel_steer" type="revolute">
+      <parent link="$(arg prefix)base_link"/>
+      <child link="$(arg prefix)rear_wheel_steer_link"/>
+      <origin xyz="-0.2899 0 0.27555" rpy="0 0 0"/>
+      <axis xyz="0 0 1" />
+      <limit velocity="9999.0" effort="9999.0" lower="${-pi*6.0}" upper="${pi*6.0}" />
+  </joint>
+  <link name="$(arg prefix)rear_wheel_steer_link">
+    <visual>
+      <origin xyz="0 0 0" rpy="0 0 0" />
+      <geometry>
+        <mesh filename="${meshes_file_direction}/rear_wheel_steer_link.stl" scale="0.001 0.001 0.001" />
+      </geometry>
+      <material name="silver">
+        <color rgba="0.75 0.75 0.75 1"/>
+      </material>
+    </visual>
+    <collision>
+      <origin xyz="0 0 0" rpy="0 0 0" />
+      <geometry>
+        <mesh filename="${meshes_file_direction}/rear_wheel_steer_link.stl" scale="0.001 0.001 0.001" />
+      </geometry>
+    </collision>
+    <inertial>
+       <origin xyz="9.802728600e-03 5.471240900e-02 -1.376533400e-01" />
+       <mass value="7.550951000e-01" />
+       <inertia ixx="2.797322900e-03" ixy="3.290833300e-05" ixz="-1.950642500e-04"
+       iyy="3.582262300e-03" iyz="2.853288400e-04"
+       izz="1.683595100e-03" />
+    </inertial>
+  </link>
+  <joint name="$(arg prefix)rear_wheel_drive" type="continuous">
+      <parent link="$(arg prefix)rear_wheel_steer_link"/>
+      <child link="$(arg prefix)rear_wheel_drive_link"/>
+      <origin xyz="0 0 -0.18905" rpy="0 0 0"/>
+      <axis xyz="0 1 0" />
+      <limit velocity="9999.0" effort="9999.0"/>
+  </joint>
+  <link name="$(arg prefix)rear_wheel_drive_link">
+    <visual>
+      <origin xyz="0 0 0" rpy="0 0 0" />
+      <geometry>
+        <mesh filename="${meshes_file_direction}/rear_wheel_drive_link.stl" scale="0.001 0.001 0.001" />
+      </geometry>
+      <material name="silver">
+        <color rgba="0.75 0.75 0.75 1"/>
+      </material>
+    </visual>
+    <collision>
+      <origin xyz="0 0 0" rpy="0 0 0" />
+      <geometry>
+        <mesh filename="${meshes_file_direction}/rear_wheel_drive_link.stl" scale="0.001 0.001 0.001" />
+      </geometry>
+    </collision>
+    <inertial>
+       <origin xyz="0.000000000e+00 1.499601700e-03 0.000000000e+00" />
+       <mass value="3.795460500e+00" />
+       <inertia ixx="7.187881500e-03" ixy="0.000000000e+00" ixz="0.000000000e+00"
+       iyy="1.156399900e-02" iyz="0.000000000e+00"
+       izz="7.187977000e-03" />
+    </inertial>
+  </link>
   <joint name="$(arg prefix)gripper_r_joint1" type="revolute">
     <parent link="$(arg prefix)base_link" />
@@ -91,4 +351,16 @@
       </visual>
   </link>
+  <xacro:ffw_sh5_follower_system
+    use_sim="$(arg use_sim)"
+    use_mock_hardware="$(arg use_mock_hardware)"
+    mock_sensor_commands="$(arg mock_sensor_commands)"/>
+  <xacro:ffw_sh5_base_system
+    use_sim="$(arg use_sim)"
+    use_mock_hardware="$(arg use_mock_hardware)"
+    mock_sensor_commands="$(arg mock_sensor_commands)"/>
+  <xacro:ffw_sh5_sensor_system
+    use_sim="$(arg use_sim)"
+    use_mock_hardware="$(arg use_mock_hardware)"
+    mock_sensor_commands="$(arg mock_sensor_commands)"/>
   <gazebo>
       <plugin filename="gz_ros2_control-system" name="gz_ros2_control::GazeboSimROS2ControlPlugin">

Commit message: Added ffw_sh5_rev1_follower bringup
Signed-off-by: Hyunwoo Nam <nhw@robotis.com>

File: ffw_description/ros2_control/ffw_sh5_rev1_follower/ffw_sh5_follower.ros2_control.xacro (robot description, xacro)
@@ -2780,37 +2780,4 @@
       </gpio>
     </ros2_control>
-    <ros2_control name="ffw_bh5_preset_hands" type="system">
-      <xacro:if value="$(arg use_sim)">
-        <hardware>
-          <plugin>gz_ros2_control/GazeboSimSystem</plugin>
-        </hardware>
-      </xacro:if>
-      <xacro:unless value="$(arg use_sim)">
-        <hardware>
-          <xacro:if value="${use_mock_hardware}">
-            <plugin>fake_components/GenericSystem</plugin>
-            <param name="mock_sensor_commands">${mock_sensor_commands}</param>
-            <param name="state_following_offset">0.0</param>
-          </xacro:if>
-          <xacro:unless value="${use_mock_hardware}">
-            <plugin>joint_state_topic_hardware_interface/JointStateTopicSystem</plugin>
-            <param name="joint_commands_topic">/topic_based_joint_commands</param>
-            <param name="joint_states_topic">/topic_based_joint_states</param>
-          </xacro:unless>
-        </hardware>
-      </xacro:unless>
-      <joint name="gripper_r_joint1">
-        <command_interface name="position"/>
-        <state_interface name="position"/>
-        <state_interface name="velocity"/>
-        <state_interface name="effort"/>
-      </joint>
-      <joint name="gripper_l_joint1">
-        <command_interface name="position"/>
-        <state_interface name="position"/>
-        <state_interface name="velocity"/>
-        <state_interface name="effort"/>
-      </joint>
-    </ros2_control>
   </xacro:macro>
 </robot>

Commit message: Renamed follower system in xacro file from ffw_sg2 to ffw_sh5 for consistency with new robot model

File: ffw_description/ros2_control/ffw_sh5_rev1_follower/ffw_sh5_follower.ros2_control.xacro (robot description, xacro)
@@ -1,6 +1,6 @@
 <?xml version="1.0"?>
 <robot xmlns:xacro="http://www.ros.org/wiki/xacro">
-  <xacro:macro name="ffw_sg2_follower_system" params="use_sim:=^|false use_mock_hardware:=^|false mock_sensor_commands:=^|false">
-    <ros2_control name="ffw_sg2_follower" type="system" is_async="true">
+  <xacro:macro name="ffw_sh5_follower_system" params="use_sim:=^|false use_mock_hardware:=^|false mock_sensor_commands:=^|false">
+    <ros2_control name="ffw_sh5_follower" type="system" is_async="true">
       <xacro:if value="$(arg use_sim)">
         <hardware>
