Commit message: Add new STL mesh files for follower components and update URDF xacro files to reference new mesh directories

File: ffw_description/urdf/ffw_bg2_rev4_follower/ffw_bg2_follower.urdf.xacro (robot description, xacro)
@@ -2,4 +2,5 @@
 <robot xmlns:xacro="http://www.ros.org/wiki/xacro" name="ffw_bg2_follower">
   <xacro:property name="meshes_file_direction" value="package://ffw_description/meshes/$(arg model)" />
+  <xacro:property name="base_meshes_dir" value="package://ffw_description/meshes/common/follower/base" />
   <xacro:arg name="use_sim" default="false" />
   <xacro:arg name="use_mock_hardware" default="false" />
@@ -22,5 +23,5 @@
       <origin xyz="0 0 0" rpy="0 0 0" />
       <geometry>
-        <mesh filename="${meshes_file_direction}/base_mobile_assy.stl" scale="0.001 0.001 0.001" />
+        <mesh filename="${base_meshes_dir}/base_mobile_assy.stl" scale="0.001 0.001 0.001" />
       </geometry>
       <material name="silver">
@@ -31,5 +32,5 @@
       <origin xyz="0 0 0" rpy="0 0 0" />
       <geometry>
-        <mesh filename="${meshes_file_direction}/base_mobile_assy.stl" scale="0.001 0.001 0.001" />
+        <mesh filename="${base_meshes_dir}/base_mobile_assy.stl" scale="0.001 0.001 0.001" />
       </geometry>
     </collision>

File: ffw_description/urdf/ffw_bh5_rev1_follower/ffw_bh5_follower.urdf.xacro (robot description, xacro)
@@ -1,5 +1,6 @@
 <?xml version="1.0"?>
 <robot xmlns:xacro="http://www.ros.org/wiki/xacro" name="ffw_bh5_follower">
-  <xacro:property name="meshes_file_direction" value="package://ffw_description/meshes/ffw_bh5_rev1_follower" />
+  <xacro:property name="meshes_file_direction" value="package://ffw_description/meshes/$(arg model)" />
+  <xacro:property name="base_meshes_dir" value="package://ffw_description/meshes/common/follower/base" />
   <xacro:arg name="use_sim" default="false" />
   <xacro:arg name="use_mock_hardware" default="false" />
@@ -24,5 +25,5 @@
       <origin xyz="0 0 0" rpy="0 0 0" />
       <geometry>
-        <mesh filename="${meshes_file_direction}/base_mobile_assy.stl" scale="0.001 0.001 0.001" />
+        <mesh filename="${base_meshes_dir}/base_mobile_assy.stl" scale="0.001 0.001 0.001" />
       </geometry>
       <material name="silver">
@@ -33,5 +34,5 @@
       <origin xyz="0 0 0" rpy="0 0 0" />
       <geometry>
-        <mesh filename="${meshes_file_direction}/base_mobile_assy.stl" scale="0.001 0.001 0.001" />
+        <mesh filename="${base_meshes_dir}/base_mobile_assy.stl" scale="0.001 0.001 0.001" />
       </geometry>
     </collision>

File: ffw_description/urdf/ffw_sg2_rev1_follower/ffw_sg2_follower.urdf.xacro (robot description, xacro)
@@ -2,4 +2,5 @@
 <robot xmlns:xacro="http://www.ros.org/wiki/xacro" name="ffw_sg2_follower">
   <xacro:property name="meshes_file_direction" value="package://ffw_description/meshes/$(arg model)" />
+  <xacro:property name="swerve_meshes_dir" value="package://ffw_description/meshes/common/follower/swerve" />
   <xacro:arg name="use_sim" default="false" />
   <xacro:arg name="use_mock_hardware" default="false" />
@@ -18,14 +19,14 @@
       <origin xyz="0 0 0" rpy="0 0 0" />
       <geometry>
-        <mesh filename="${meshes_file_direction}/base_mobile_assy.stl" scale="0.001 0.001 0.001" />
-      </geometry>
-      <material name="silver">
-        <color rgba="0.75 0.75 0.75 1"/>
-      </material>
-    </visual>
-    <collision>
-      <origin xyz="0 0 0" rpy="0 0 0" />
-      <geometry>
-        <mesh filename="${meshes_file_direction}/base_mobile_assy.stl" scale="0.001 0.001 0.001" />
+        <mesh filename="${swerve_meshes_dir}/base_mobile_assy.stl" scale="0.001 0.001 0.001" />
+      </geometry>
+      <material name="silver">
+        <color rgba="0.75 0.75 0.75 1"/>
+      </material>
+    </visual>
+    <collision>
+      <origin xyz="0 0 0" rpy="0 0 0" />
+      <geometry>
+        <mesh filename="${swerve_meshes_dir}/base_mobile_assy.stl" scale="0.001 0.001 0.001" />
       </geometry>
     </collision>
@@ -86,14 +87,14 @@
       <origin xyz="0 0 0" rpy="0 0 0" />
       <geometry>
-        <mesh filename="${meshes_file_direction}/lift_link.stl" scale="0.001 0.001 0.001" />
-      </geometry>
-      <material name="silver">
-        <color rgba="0.75 0.75 0.75 1"/>
-      </material>
-    </visual>
-    <collision>
-      <origin xyz="0 0 0" rpy="0 0 0" />
-      <geometry>
-        <mesh filename="${meshes_file_direction}/lift_link.stl" scale="0.001 0.001 0.001" />
+        <mesh filename="${swerve_meshes_dir}/lift_link.stl" scale="0.001 0.001 0.001" />
+      </geometry>
+      <material name="silver">
+        <color rgba="0.75 0.75 0.75 1"/>
+      </material>
+    </visual>
+    <collision>
+      <origin xyz="0 0 0" rpy="0 0 0" />
+      <geometry>
+        <mesh filename="${swerve_meshes_dir}/lift_link.stl" scale="0.001 0.001 0.001" />
       </geometry>
     </collision>
@@ -165,14 +166,14 @@
       <origin xyz="0 0 0" rpy="0 0 0" />
       <geometry>
-        <mesh filename="${meshes_file_direction}/left_wheel_steer_link.stl" scale="0.001 0.001 0.001" />
-      </geometry>
-      <material name="silver">
-        <color rgba="0.75 0.75 0.75 1"/>
-      </material>
-    </visual>
-    <collision>
-      <origin xyz="0 0 0" rpy="0 0 0" />
-      <geometry>
-        <mesh filename="${meshes_file_direction}/left_wheel_steer_link.stl" scale="0.001 0.001 0.001" />
+        <mesh filename="${swerve_meshes_dir}/left_wheel_steer_link.stl" scale="0.001 0.001 0.001" />
+      </geometry>
+      <material name="silver">
+        <color rgba="0.75 0.75 0.75 1"/>
+      </material>
+    </visual>
+    <collision>
+      <origin xyz="0 0 0" rpy="0 0 0" />
+      <geometry>
+        <mesh filename="${swerve_meshes_dir}/left_wheel_steer_link.stl" scale="0.001 0.001 0.001" />
       </geometry>
     </collision>
@@ -196,5 +197,5 @@
       <origin xyz="0 0 0" rpy="0 0 0" />
       <geometry>
-        <mesh filename="${meshes_file_direction}/left_wheel_drive_link.stl" scale="0.001 0.001 0.001" />
+        <mesh filename="${swerve_meshes_dir}/left_wheel_drive_link.stl" scale="0.001 0.001 0.001" />
       </geometry>
       <material name="silver">
@@ -205,5 +206,5 @@
       <origin xyz="0 0 0" rpy="0 0 0" />
       <geometry>
-        <mesh filename="${meshes_file_direction}/left_wheel_drive_link.stl" scale="0.001 0.001 0.001" />
+        <mesh filename="${swerve_meshes_dir}/left_wheel_drive_link.stl" scale="0.001 0.001 0.001" />
       </geometry>
     </collision> -->
@@ -233,14 +234,14 @@
       <origin xyz="0 0 0" rpy="0 0 0" />
       <geometry>
-        <mesh filename="${meshes_file_direction}/right_wheel_steer_link.stl" scale="0.001 0.001 0.001" />
-      </geometry>
-      <material name="silver">
-        <color rgba="0.75 0.75 0.75 1"/>
-      </material>
-    </visual>
-    <collision>
-      <origin xyz="0 0 0" rpy="0 0 0" />
-      <geometry>
-        <mesh filename="${meshes_file_direction}/right_wheel_steer_link.stl" scale="0.001 0.001 0.001" />
+        <mesh filename="${swerve_meshes_dir}/right_wheel_steer_link.stl" scale="0.001 0.001 0.001" />
+      </geometry>
+      <material name="silver">
+        <color rgba="0.75 0.75 0.75 1"/>
+      </material>
+    </visual>
+    <collision>
+      <origin xyz="0 0 0" rpy="0 0 0" />
+      <geometry>
+        <mesh filename="${swerve_meshes_dir}/right_wheel_steer_link.stl" scale="0.001 0.001 0.001" />
       </geometry>
     </collision>
@@ -264,5 +265,5 @@
       <origin xyz="0 0 0" rpy="0 0 0" />
       <geometry>
-        <mesh filename="${meshes_file_direction}/right_wheel_drive_link.stl" scale="0.001 0.001 0.001" />
+        <mesh filename="${swerve_meshes_dir}/right_wheel_drive_link.stl" scale="0.001 0.001 0.001" />
       </geometry>
       <material name="silver">
@@ -273,5 +274,5 @@
       <origin xyz="0 0 0" rpy="0 0 0" />
       <geometry>
-        <mesh filename="${meshes_file_direction}/right_wheel_drive_link.stl" scale="0.001 0.001 0.001" />
+        <mesh filename="${swerve_meshes_dir}/right_wheel_drive_link.stl" scale="0.001 0.001 0.001" />
       </geometry>
     </collision> -->
@@ -301,14 +302,14 @@
       <origin xyz="0 0 0" rpy="0 0 0" />
       <geometry>
-        <mesh filename="${meshes_file_direction}/rear_wheel_steer_link.stl" scale="0.001 0.001 0.001" />
-      </geometry>
-      <material name="silver">
-        <color rgba="0.75 0.75 0.75 1"/>
-      </material>
-    </visual>
-    <collision>
-      <origin xyz="0 0 0" rpy="0 0 0" />
-      <geometry>
-        <mesh filename="${meshes_file_direction}/rear_wheel_steer_link.stl" scale="0.001 0.001 0.001" />
+        <mesh filename="${swerve_meshes_dir}/rear_wheel_steer_link.stl" scale="0.001 0.001 0.001" />
+      </geometry>
+      <material name="silver">
+        <color rgba="0.75 0.75 0.75 1"/>
+      </material>
+    </visual>
+    <collision>
+      <origin xyz="0 0 0" rpy="0 0 0" />
+      <geometry>
+        <mesh filename="${swerve_meshes_dir}/rear_wheel_steer_link.stl" scale="0.001 0.001 0.001" />
       </geometry>
     </collision>
@@ -332,5 +333,5 @@
       <origin xyz="0 0 0" rpy="0 0 0" />
       <geometry>
-        <mesh filename="${meshes_file_direction}/rear_wheel_drive_link.stl" scale="0.001 0.001 0.001" />
+        <mesh filename="${swerve_meshes_dir}/rear_wheel_drive_link.stl" scale="0.001 0.001 0.001" />
       </geometry>
       <material name="silver">
@@ -347,5 +348,5 @@
       <origin xyz="0 0 0" rpy="0 0 0" />
       <geometry>
-        <mesh filename="${meshes_file_direction}/rear_wheel_drive_link.stl" scale="0.001 0.001 0.001" />
+        <mesh filename="${swerve_meshes_dir}/rear_wheel_drive_link.stl" scale="0.001 0.001 0.001" />
       </geometry>
     </collision> -->

File: ffw_description/urdf/ffw_sh5_rev1_follower/ffw_sh5_follower.urdf.xacro (robot description, xacro)
@@ -2,4 +2,5 @@
 <robot xmlns:xacro="http://www.ros.org/wiki/xacro" name="ffw_sh5_follower">
   <xacro:property name="meshes_file_direction" value="package://ffw_description/meshes/$(arg model)" />
+  <xacro:property name="swerve_meshes_dir" value="package://ffw_description/meshes/common/follower/swerve" />
   <xacro:arg name="use_sim" default="false" />
   <xacro:arg name="use_mock_hardware" default="false" />
@@ -18,14 +19,14 @@
       <origin xyz="0 0 0" rpy="0 0 0" />
       <geometry>
-        <mesh filename="${meshes_file_direction}/base_mobile_assy.stl" scale="0.001 0.001 0.001" />
-      </geometry>
-      <material name="silver">
-        <color rgba="0.75 0.75 0.75 1"/>
-      </material>
-    </visual>
-    <collision>
-      <origin xyz="0 0 0" rpy="0 0 0" />
-      <geometry>
-        <mesh filename="${meshes_file_direction}/base_mobile_assy.stl" scale="0.001 0.001 0.001" />
+        <mesh filename="${swerve_meshes_dir}/base_mobile_assy.stl" scale="0.001 0.001 0.001" />
+      </geometry>
+      <material name="silver">
+        <color rgba="0.75 0.75 0.75 1"/>
+      </material>
+    </visual>
+    <collision>
+      <origin xyz="0 0 0" rpy="0 0 0" />
+      <geometry>
+        <mesh filename="${swerve_meshes_dir}/base_mobile_assy.stl" scale="0.001 0.001 0.001" />
       </geometry>
     </collision>
@@ -64,14 +65,14 @@
       <origin xyz="0 0 0" rpy="0 0 0" />
       <geometry>
-        <mesh filename="${meshes_file_direction}/lift_link.stl" scale="0.001 0.001 0.001" />
-      </geometry>
-      <material name="silver">
-        <color rgba="0.75 0.75 0.75 1"/>
-      </material>
-    </visual>
-    <collision>
-      <origin xyz="0 0 0" rpy="0 0 0" />
-      <geometry>
-        <mesh filename="${meshes_file_direction}/lift_link.stl" scale="0.001 0.001 0.001" />
+        <mesh filename="${swerve_meshes_dir}/lift_link.stl" scale="0.001 0.001 0.001" />
+      </geometry>
+      <material name="silver">
+        <color rgba="0.75 0.75 0.75 1"/>
+      </material>
+    </visual>
+    <collision>
+      <origin xyz="0 0 0" rpy="0 0 0" />
+      <geometry>
+        <mesh filename="${swerve_meshes_dir}/lift_link.stl" scale="0.001 0.001 0.001" />
       </geometry>
     </collision>
@@ -109,14 +110,14 @@
       <origin xyz="0 0 0" rpy="0 0 0" />
       <geometry>
-        <mesh filename="${meshes_file_direction}/left_wheel_steer_link.stl" scale="0.001 0.001 0.001" />
-      </geometry>
-      <material name="silver">
-        <color rgba="0.75 0.75 0.75 1"/>
-      </material>
-    </visual>
-    <collision>
-      <origin xyz="0 0 0" rpy="0 0 0" />
-      <geometry>
-        <mesh filename="${meshes_file_direction}/left_wheel_steer_link.stl" scale="0.001 0.001 0.001" />
+        <mesh filename="${swerve_meshes_dir}/left_wheel_steer_link.stl" scale="0.001 0.001 0.001" />
+      </geometry>
+      <material name="silver">
+        <color rgba="0.75 0.75 0.75 1"/>
+      </material>
+    </visual>
+    <collision>
+      <origin xyz="0 0 0" rpy="0 0 0" />
+      <geometry>
+        <mesh filename="${swerve_meshes_dir}/left_wheel_steer_link.stl" scale="0.001 0.001 0.001" />
       </geometry>
     </collision>
@@ -140,5 +141,5 @@
       <origin xyz="0 0 0" rpy="0 0 0" />
       <geometry>
-        <mesh filename="${meshes_file_direction}/left_wheel_drive_link.stl" scale="0.001 0.001 0.001" />
+        <mesh filename="${swerve_meshes_dir}/left_wheel_drive_link.stl" scale="0.001 0.001 0.001" />
       </geometry>
       <material name="silver">
@@ -149,5 +150,5 @@
       <origin xyz="0 0 0" rpy="0 0 0" />
       <geometry>
-        <mesh filename="${meshes_file_direction}/left_wheel_drive_link.stl" scale="0.001 0.001 0.001" />
+        <mesh filename="${swerve_meshes_dir}/left_wheel_drive_link.stl" scale="0.001 0.001 0.001" />
       </geometry>
     </collision> -->
@@ -177,14 +178,14 @@
       <origin xyz="0 0 0" rpy="0 0 0" />
       <geometry>
-        <mesh filename="${meshes_file_direction}/right_wheel_steer_link.stl" scale="0.001 0.001 0.001" />
-      </geometry>
-      <material name="silver">
-        <color rgba="0.75 0.75 0.75 1"/>
-      </material>
-    </visual>
-    <collision>
-      <origin xyz="0 0 0" rpy="0 0 0" />
-      <geometry>
-        <mesh filename="${meshes_file_direction}/right_wheel_steer_link.stl" scale="0.001 0.001 0.001" />
+        <mesh filename="${swerve_meshes_dir}/right_wheel_steer_link.stl" scale="0.001 0.001 0.001" />
+      </geometry>
+      <material name="silver">
+        <color rgba="0.75 0.75 0.75 1"/>
+      </material>
+    </visual>
+    <collision>
+      <origin xyz="0 0 0" rpy="0 0 0" />
+      <geometry>
+        <mesh filename="${swerve_meshes_dir}/right_wheel_steer_link.stl" scale="0.001 0.001 0.001" />
       </geometry>
     </collision>
@@ -208,5 +209,5 @@
       <origin xyz="0 0 0" rpy="0 0 0" />
       <geometry>
-        <mesh filename="${meshes_file_direction}/right_wheel_drive_link.stl" scale="0.001 0.001 0.001" />
+        <mesh filename="${swerve_meshes_dir}/right_wheel_drive_link.stl" scale="0.001 0.001 0.001" />
       </geometry>
       <material name="silver">
@@ -217,5 +218,5 @@
       <origin xyz="0 0 0" rpy="0 0 0" />
       <geometry>
-        <mesh filename="${meshes_file_direction}/right_wheel_drive_link.stl" scale="0.001 0.001 0.001" />
+        <mesh filename="${swerve_meshes_dir}/right_wheel_drive_link.stl" scale="0.001 0.001 0.001" />
       </geometry>
     </collision> -->
@@ -245,14 +246,14 @@
       <origin xyz="0 0 0" rpy="0 0 0" />
       <geometry>
-        <mesh filename="${meshes_file_direction}/rear_wheel_steer_link.stl" scale="0.001 0.001 0.001" />
-      </geometry>
-      <material name="silver">
-        <color rgba="0.75 0.75 0.75 1"/>
-      </material>
-    </visual>
-    <collision>
-      <origin xyz="0 0 0" rpy="0 0 0" />
-      <geometry>
-        <mesh filename="${meshes_file_direction}/rear_wheel_steer_link.stl" scale="0.001 0.001 0.001" />
+        <mesh filename="${swerve_meshes_dir}/rear_wheel_steer_link.stl" scale="0.001 0.001 0.001" />
+      </geometry>
+      <material name="silver">
+        <color rgba="0.75 0.75 0.75 1"/>
+      </material>
+    </visual>
+    <collision>
+      <origin xyz="0 0 0" rpy="0 0 0" />
+      <geometry>
+        <mesh filename="${swerve_meshes_dir}/rear_wheel_steer_link.stl" scale="0.001 0.001 0.001" />
       </geometry>
     </collision>
@@ -276,5 +277,5 @@
       <origin xyz="0 0 0" rpy="0 0 0" />
       <geometry>
-        <mesh filename="${meshes_file_direction}/rear_wheel_drive_link.stl" scale="0.001 0.001 0.001" />
+        <mesh filename="${swerve_meshes_dir}/rear_wheel_drive_link.stl" scale="0.001 0.001 0.001" />
       </geometry>
       <material name="silver">
@@ -285,5 +286,5 @@
       <origin xyz="0 0 0" rpy="0 0 0" />
       <geometry>
-        <mesh filename="${meshes_file_direction}/rear_wheel_drive_link.stl" scale="0.001 0.001 0.001" />
+        <mesh filename="${swerve_meshes_dir}/rear_wheel_drive_link.stl" scale="0.001 0.001 0.001" />
       </geometry>
     </collision> -->
